File: KiCAD/PCB projet ESE/PCB projet ESE.kicad_pcb (KiCad board)
At the start: 2 copper layers, 57 x 54 mm, 126 parts, among them J1 Conn_01x06, J10 Conn_01x06, J11 Conn_01x06, J12 Conn_01x04, J13 Conn_01x02, J14 Conn_01x03, J15 Conn_01x04, J16 Conn_01x06, J17 Conn_01x03, J18 Conn_01x03, J19 Conn_01x03, J2 Conn_01x06, J20 Conn_01x03, J21 Conn_01x03, J22 Conn_01x03, J23 Conn_01x03, J24 Conn_01x03, J25 Conn_01x03, J26 Conn_01x03, J27 Conn_01x03, J28 Conn_01x03, J29 USB_C_Receptacle_USB2.0_16P, J3 Conn_01x06, J4 Conn_01x06, J5 Conn_01x06, J6 Conn_01x06, J7 Conn_01x06, J8 Conn_01x06, J9 Conn_ST_STDC14, SW1 SW_SPST, SW2 SW_SPDT, U1 STM32G474RETx, U2 ADXL343, U3 ZXBM5210-SP, U4 ZXBM5210-SP, U5 USBLC6-2SC6

Commit message: PCB
Parts:
- removed C10A1, C1A1, C1A2, C2A1, C2A2, C7A1: 22u, Capacitor_SMD:C_Elec_5x5.4
- removed MP4, MP5: ~, Régu:TSOT23-8
- added C35: 0.1u, Capacitor_SMD:C_0402_1005Metric, F.Cu at (192.1, 83.1)
- added C36: 0.1u, Capacitor_SMD:C_0402_1005Metric, F.Cu at (192.1, 85.1)
- added C37: 0.1u, Capacitor_SMD:C_0402_1005Metric, F.Cu at (192.1, 87.0)
- added C38: 15p, Capacitor_SMD:C_0402_1005Metric, F.Cu at (192.1, 89.0)
- added C39: 22u, Capacitor_SMD:C_Elec_5x5.4, F.Cu at (196.8, 71.8)
- added C40: 22u, Capacitor_SMD:C_Elec_5x5.4, F.Cu at (196.8, 78.7)
- added MP1: ~, Régu:TSOT23-8, F.Cu at (178.3, 84.3)
- added MP2: ~, Régu:TSOT23-8, F.Cu at (178.3, 88.5)
- C1: value 4u7 -> 100n; footprint Capacitor_SMD:C_0603_1608Metric -> Capacitor_SMD:C_0402_1005Metric
- C10, C8: value 1u -> 100n; footprint Capacitor_SMD:C_0603_1608Metric -> Capacitor_SMD:C_0402_1005Metric
- C11, C13: value 0.1u -> 100n
- C14: value 100n -> 10n
- C15, C18: value 4.7u -> 1u
- C17: value 100n -> 0.1u
- C19, C20, C30, C31: value 0.1u -> 22u; footprint Capacitor_SMD:C_0402_1005Metric -> Capacitor_SMD:C_Elec_5x5.4
- C2, C5: value 100n -> 4.7u; footprint Capacitor_SMD:C_0402_1005Metric -> Capacitor_SMD:C_0603_1608Metric
- C22: value 1u -> 0.1u; footprint Capacitor_SMD:C_0603_1608Metric -> Capacitor_SMD:C_0402_1005Metric
- C25: value 15p -> 1u; footprint Capacitor_SMD:C_0402_1005Metric -> Capacitor_SMD:C_0603_1608Metric
- C26: value 15p -> 0.1u
- C27: value 22u -> 0.1u; footprint Capacitor_SMD:C_Elec_5x5.4 -> Capacitor_SMD:C_0402_1005Metric
- C28: value 22u -> 15p; footprint Capacitor_SMD:C_Elec_5x5.4 -> Capacitor_SMD:C_0402_1005Metric
- C29: value 0.1u -> 15p
- C32: value 15p -> 22u; footprint Capacitor_SMD:C_0402_1005Metric -> Capacitor_SMD:C_Elec_5x5.4
- C34: value 100n -> 22u; footprint Capacitor_SMD:C_0402_1005Metric -> Capacitor_SMD:C_Elec_5x5.4
- C6: value 1u -> 4u7
- C9: value 10n -> 1u; footprint Capacitor_SMD:C_0402_1005Metric -> Capacitor_SMD:C_0603_1608Metric
- J12, J15: value Conn_01x04 -> Conn_01x06; footprint Connector_JST:JST_PH_B4B-PH-K_1x04_P2.00mm_Vertical -> Connector_JST:JST_PH_B6B-PH-K_1x06_P2.00mm_Vertical
- J13: value Conn_01x02 -> Conn_01x06; footprint Connector_AMASS:AMASS_XT60-M_1x02_P7.20mm_Vertical -> Connector_JST:JST_PH_B6B-PH-K_1x06_P2.00mm_Vertical
- J14: value Conn_01x03 -> Conn_01x06; footprint Connector_JST:JST_PH_B3B-PH-K_1x03_P2.00mm_Vertical -> Connector_JST:JST_PH_B6B-PH-K_1x06_P2.00mm_Vertical
- J16: value Conn_01x06 -> Conn_01x03; footprint Connector_JST:JST_PH_B6B-PH-K_1x06_P2.00mm_Vertical -> Connector_JST:JST_PH_B3B-PH-K_1x03_P2.00mm_Vertical
- J2, J6: value Conn_01x06 -> Conn_01x04; footprint Connector_JST:JST_PH_B6B-PH-K_1x06_P2.00mm_Vertical -> Connector_JST:JST_PH_B4B-PH-K_1x04_P2.00mm_Vertical
- J5: value Conn_01x06 -> Conn_01x02; footprint Connector_JST:JST_PH_B6B-PH-K_1x06_P2.00mm_Vertical -> Connector_AMASS:AMASS_XT60-M_1x02_P7.20mm_Vertical
- J7: value Conn_01x06 -> Conn_ST_STDC14; footprint Connector_JST:JST_PH_B6B-PH-K_1x06_P2.00mm_Vertical -> Connector_PinHeader_1.27mm:PinHeader_2x07_P1.27mm_Vertical_SMD
- J9: value Conn_ST_STDC14 -> Conn_01x06; footprint Connector_PinHeader_1.27mm:PinHeader_2x07_P1.27mm_Vertical_SMD -> Connector_JST:JST_PH_B6B-PH-K_1x06_P2.00mm_Vertical
- L1: footprint Capacitor_SMD:C_0402_1005Metric_Pad0.74x0.62mm_HandSolder -> Inductor_SMD:L_0603_1608Metric
- R1: value 1k -> 47k
- R10, R11: value 5k1 -> 1k
- R2: value 1k -> 10k
- R3: value 1k -> 6k55
- R30: value 47k -> 5k1
- R31: value 10k -> 5k1
- R4: value 1k -> 2k9
- R5: value 6k55 -> 1k65
- R6: value 2k9 -> 1k
- R7: value 1k65 -> 800
- R8: value 800 -> 1k
- SW2: value SW_SPDT -> 472121010111; footprint Régu:SW_SPDT -> Régu:SW_Wurth_WS-TOTV_472123020421
- U1: value STM32G474RETx -> ZXBM5210-SP; footprint Package_QFP:LQFP-64_10x10mm_P0.5mm -> Package_SO:Diodes_SO-8EP
- U2: value ADXL343 -> ZXBM5210-SP; footprint Package_LGA:LGA-14_3x5mm_P0.8mm_LayoutBorder1x6y -> Package_SO:Diodes_SO-8EP
- U3: value ZXBM5210-SP -> STM32G474RETx; footprint Package_SO:Diodes_SO-8EP -> Package_QFP:LQFP-64_10x10mm_P0.5mm
- U4: value ZXBM5210-SP -> ADXL343; footprint Package_SO:Diodes_SO-8EP -> Package_LGA:LGA-14_3x5mm_P0.8mm_LayoutBorder1x6y
- moved R10 146.2 mm to (115.3, 71.5), turned to 180 degrees
- moved R11 146.0 mm to (115.3, 72.5), turned to 180 degrees
- moved C3 137.4 mm to (91.3, 77.4)
- moved R1 133.6 mm to (91.5, 73.0)
- moved R2 133.6 mm to (91.5, 75.0)
- moved C14 129.0 mm to (101.5, 67.7), turned to 90 degrees
- moved H4 128.5 mm to (84.0, 95.0)
- moved C2 128.2 mm to (133.2, 145.0)
- moved C7 127.4 mm to (100.2, 71.5), turned to 90 degrees
- moved H1 126.1 mm to (84.0, 51.0)
- moved C5 125.9 mm to (133.2, 147.5)
- moved C1 125.5 mm to (134.0, 138.3)
- moved C4 123.2 mm to (134.0, 142.2)
- moved C11 123.2 mm to (109.3, 80.2), turned to 180 degrees
- moved U1 122.4 mm to (142.5, 139.5)
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Connections:
- BUxxSD1 pad 1: (no net) -> +5V
- BUxxSD1 pad 2: (no net) -> GND
- BUxxSD1 pad 4: (no net) -> unconnected-(BUxxSD1-NC-Pad4)
- BUxxSD1 pad 5: (no net) -> +3.3V
- C1 pad 1: +3.3V -> +7.5V
- C12 pad 1: NRST -> +3.3V
- C13 pad 1: Net-(MP4-VCC) -> +3.3V
- C14 pad 1: +7.5V -> +3.3V
- C15 pad 1: GND -> unconnected-(C15-Pad1)
- C15 pad 2: +7.5V -> unconnected-(C15-Pad2)
- C16 pad 1: +5V -> GND
- C16 pad 2: GND -> +3.3V
- C17 pad 1: +7.5V -> +3.3V
- C18 pad 1: GND -> +5V
- C18 pad 2: +7.5V -> GND
- C19 pad 1: Net-(MP3-VCC) -> GND
- C19 pad 2: GND -> +14.8V
- C2 pad 1: +3.3V -> GND
- C2 pad 2: GND -> +7.5V
- C21 pad 1: GND -> Net-(MP1-VCC)
- C21 pad 2: +14.8V -> GND
- C22 pad 1: +3.3V -> Net-(MP2-VCC)
- C23 pad 1: Net-(C23-Pad1) -> GND
- C23 pad 2: Net-(MP4-SW) -> +14.8V
- C24 pad 1: Net-(C24-Pad1) -> GND
- C24 pad 2: Net-(MP3-SW) -> +14.8V
- C25 pad 1: Net-(C25-Pad1) -> +3.3V
- C25 pad 2: +5V -> GND
- C26 pad 2: +7.5V -> Net-(MP1-SW)
- C27 pad 1: GND -> Net-(C27-Pad1)
- C27 pad 2: +5V -> Net-(MP2-SW)
- C28 pad 1: GND -> Net-(C28-Pad1)
- C28 pad 2: +7.5V -> +5V
- C29 pad 1: Net-(MP5-VCC) -> Net-(C29-Pad1)
- C29 pad 2: GND -> +7.5V
- C3 pad 1: +3.3V -> ADC
- C30 pad 2: +14.8V -> +5V
- C31 pad 1: Net-(C31-Pad1) -> GND
- C31 pad 2: Net-(MP5-SW) -> +7.5V
- C32 pad 1: Net-(C32-Pad1) -> GND
- C32 pad 2: +2.8V -> +5V
- C33 pad 2: +2.8V -> +7.5V
- C34 pad 1: ADC -> GND
- C34 pad 2: GND -> +14.8V
- C4 pad 1: +3.3V -> +7.5V
- C5 pad 1: +3.3V -> GND
- C5 pad 2: GND -> +7.5V
- C7 pad 1: +3.3V -> NRST
- C8 pad 1: GND -> +3.3V
- C8 pad 2: +3.3V -> GND
- J1 pad 1: INT -> GND
- J1 pad 2: SCL TOF -> GND
- J1 pad 3: XSHUT_1 -> Encodeur phase A 1
- J1 pad 4: SDA TOF -> Encodeur Phase B 1
- J1 pad 5: +2.8V -> +3.3V
- J1 pad 6: GND -> +7.5V
- J10 pad 3: XSHUT_3 -> XSHUT_7
- J11 pad 3: XSHUT_6 -> XSHUT_2
- J12 pad 1: +3.3V -> INT
- J12 pad 2: GND -> SCL TOF
- J12 pad 3: Lidar Output  -> XSHUT_5
- J12 pad 4: +5V -> SDA TOF
- J13 pad 1: GND -> INT
- J13 pad 2: Net-(J13-Pin_2) -> SCL TOF
- J14 pad 1: GND -> INT
- J14 pad 2: PWM_LED1 -> SCL TOF
- J14 pad 3: +5V -> XSHUT_3
- J15 pad 1: UART_mp3_RX -> INT
- J15 pad 2: UART_mp3_TX -> SCL TOF
- J15 pad 3: +5V -> XSHUT_6
- J15 pad 4: GND -> SDA TOF
- J16 pad 1: unconnected-(J16-Pin_1-Pad1) -> GND
- J16 pad 2: +5V -> PWM_LED1
- J16 pad 3: GND -> +5V
- J17 pad 2: PWM_LED2 -> PWM_LED4
- J18 pad 2: PWM_LED3 -> PWM_LED2
- J19 pad 2: PWM_LED4 -> PWM_LED5
- J2 pad 1: INT -> UART_mp3_RX
- J2 pad 2: SCL TOF -> UART_mp3_TX
- J2 pad 3: XSHUT_2 -> +5V
- J2 pad 4: SDA TOF -> GND
- J20 pad 2: PWM_LED5 -> PWM_LED3
- J3 pad 1: INT -> GND
- J3 pad 2: SCL TOF -> GND
- J3 pad 3: XSHUT_4 -> Encodeur phase A 2
- J3 pad 4: SDA TOF -> Encodeur Phase B 2
- J3 pad 5: +2.8V -> +3.3V
- J3 pad 6: GND -> +7.5V
- J4 pad 1: INT -> unconnected-(J4-Pin_1-Pad1)
- J4 pad 2: SCL TOF -> +5V
- J4 pad 3: XSHUT_5 -> GND
- J4 pad 4: SDA TOF -> UART_HC05_TX
- J4 pad 5: +2.8V -> UART_HC05_RX
- J4 pad 6: GND -> unconnected-(J4-Pin_6-Pad6)
- J5 pad 2: GND -> Net-(J5-Pin_2)
- J6 pad 1: GND -> +3.3V
- J6 pad 3: Encodeur phase A 2 -> Lidar Output 
- J6 pad 4: Encodeur Phase B 2 -> +5V
- J7 pad 1: INT -> unconnected-(J7-NC-Pad1)
- J7 pad 2: SCL TOF -> unconnected-(J7-NC-Pad2)
- J7 pad 3: XSHUT_7 -> +3.3V
- J7 pad 4: SDA TOF -> SWDIO
- J7 pad 5: +2.8V -> GND
- J7 pad 6: GND -> SWCLK
- J8 pad 3: XSHUT_8 -> XSHUT_1
- J9 pad 1: unconnected-(J9-NC-Pad1) -> INT
- J9 pad 2: unconnected-(J9-NC-Pad2) -> SCL TOF
- J9 pad 3: +3.3V -> XSHUT_4
- J9 pad 4: SWDIO -> SDA TOF
- J9 pad 5: GND -> +2.8V
- J9 pad 6: SWCLK -> GND
- L2 pad 1: Net-(MP4-SW) -> Net-(MP1-SW)
- L3 pad 1: Net-(MP3-SW) -> Net-(MP2-SW)
- L4 pad 1: Net-(MP5-SW) -> Net-(MP3-SW)
- MP3 pad 1: (no net) -> PG_2.8
- MP3 pad 2: (no net) -> +14.8V
- MP3 pad 3: (no net) -> Net-(MP3-SW)
- MP3 pad 4: (no net) -> GND
- MP3 pad 5: (no net) -> Net-(MP3-BST)
- MP3 pad 6: (no net) -> EN/SYNC_2.8
- MP3 pad 7: (no net) -> Net-(MP3-VCC)
- MP3 pad 8: (no net) -> Net-(MP3-FB)
- R1 pad 1: +3.3V -> +14.8V
- R1 pad 2: Accel SDA -> ADC
- R10 pad 1: Net-(J29-CC1) -> +3.3V
- R10 pad 2: GND -> SDA TOF
- R11 pad 1: Net-(J29-CC2) -> +3.3V
- R11 pad 2: GND -> SCL TOF
- R14 pad 1: Net-(MP4-VCC) -> Net-(MP1-VCC)
- R15 pad 1: Net-(MP3-VCC) -> Net-(MP2-VCC)
- R16 pad 2: Net-(C23-Pad1) -> Net-(C26-Pad1)
- R17 pad 2: Net-(C24-Pad1) -> Net-(C27-Pad1)
- R18 pad 1: Net-(C25-Pad1) -> Net-(C28-Pad1)
- R19 pad 1: Net-(C26-Pad1) -> Net-(C29-Pad1)
- R2 pad 1: +3.3V -> ADC
- R2 pad 2: Accel SCL -> GND
- R20 pad 1: Net-(C25-Pad1) -> Net-(C28-Pad1)
- R21 pad 1: Net-(C26-Pad1) -> Net-(C29-Pad1)
- R22 pad 1: Net-(C25-Pad1) -> Net-(C28-Pad1)
- R23 pad 1: Net-(C26-Pad1) -> Net-(C29-Pad1)
- R25 pad 1: Net-(MP5-VCC) -> Net-(MP3-VCC)
- R26 pad 1: Net-(MP5-BST) -> Net-(MP3-BST)
- R26 pad 2: Net-(C31-Pad1) -> Net-(C37-Pad1)
- R27 pad 1: Net-(C32-Pad1) -> Net-(C38-Pad1)
- R27 pad 2: Net-(MP5-FB) -> Net-(MP3-FB)
- R28 pad 1: Net-(C32-Pad1) -> Net-(C38-Pad1)
- R29 pad 1: Net-(C32-Pad1) -> Net-(C38-Pad1)
- R3 pad 1: +3.3V -> +14.8V
- R3 pad 2: SDA TOF -> Net-(D1-A)
- R30 pad 1: +14.8V -> Net-(J29-CC1)
- R30 pad 2: ADC -> GND
- R31 pad 1: ADC -> Net-(J29-CC2)
- R4 pad 1: +3.3V -> +7.5V
- R4 pad 2: SCL TOF -> Net-(D2-A)
- R5 pad 1: +14.8V -> +5V
- R5 pad 2: Net-(D5-A) -> Net-(D3-A)
- R6 pad 1: +7.5V -> +3.3V
- R6 pad 2: Net-(D3-A) -> Accel SDA
- R7 pad 1: +5V -> +3.3V
- R8 pad 2: Net-(D2-A) -> Accel SCL
- R9 pad 2: Net-(D1-A) -> Net-(D5-A)
- SW2 pad 2: Net-(J13-Pin_2) -> Net-(J5-Pin_2)
- U1 pad 1: +3.3V -> Encodeur phase A 1
- U1 pad 2: unconnected-(U1-PC13-Pad2) -> +7.5V
- U1 pad 3: unconnected-(U1-PC14-Pad3) -> +7.5V
- U1 pad 4: unconnected-(U1-PC15-Pad4) -> PWM FWD 1
- U1 pad 5: unconnected-(U1-PF0-Pad5) -> PWM REV 1
- U1 pad 6: unconnected-(U1-PF1-Pad6) -> +7.5V
- U1 pad 7: NRST -> Encodeur Phase B 1
- U1 pad 8: PWM_servo_1 -> GND
- U1 pad 9: PWM_servo_2 -> GND
- U2 pad 1: +3.3V -> Encodeur phase A 2
- U2 pad 2: GND -> +7.5V
- U2 pad 3: unconnected-(U2-RES-Pad3) -> +7.5V
- U2 pad 4: GND -> PWM FWD 2
- U2 pad 5: GND -> PWM REV 2
- U2 pad 6: +3.3V -> +7.5V
- U2 pad 7: +3.3V -> Encodeur Phase B 2
- U2 pad 8: INT 1 -> GND
- U2 pad 9: INT 2 -> GND
- U3 pad 1: Encodeur phase A 1 -> +3.3V
- U3 pad 2: +7.5V -> unconnected-(U3-PC13-Pad2)
- U3 pad 3: +7.5V -> unconnected-(U3-PC14-Pad3)
- U3 pad 4: PWM FWD 1 -> unconnected-(U3-PC15-Pad4)
- U3 pad 5: PWM REV 1 -> unconnected-(U3-PF0-Pad5)
- U3 pad 6: +7.5V -> unconnected-(U3-PF1-Pad6)
- U3 pad 7: Encodeur Phase B 1 -> NRST
- U3 pad 8: GND -> PWM_servo_1
- U3 pad 9: GND -> PWM_servo_2
- U4 pad 1: Encodeur phase A 2 -> +3.3V
- U4 pad 2: +7.5V -> GND
- U4 pad 3: +7.5V -> unconnected-(U4-RES-Pad3)
- U4 pad 4: PWM FWD 2 -> GND
- U4 pad 5: PWM REV 2 -> GND
- U4 pad 6: +7.5V -> +3.3V
- U4 pad 7: Encodeur Phase B 2 -> +3.3V
- U4 pad 8: GND -> INT 1
- U4 pad 9: GND -> INT 2
Routing:
- added copper zone on B.Cu, net GND
- added copper zone on F.Cu, net GND
- added copper zone on In1.Cu, net GND
Other:
- outline, holes or cut-outs redrawn
- copper layers 2 -> 4
