File: KiCAD/PCB projet ESE/Rasbpi.kicad_sch (KiCad schematic)
At the start: 4 parts, among them J29 USB_C_Receptacle_USB2.0_16P, U5 USBLC6-2SC6

Commit message: finish first version of schematic
Parts:
- added F1: 250mA, Fuse:Fuse_1206_3216Metric, symbol Device:Polyfuse_Small
- added FB1: 600 @ 100MHz, Inductor_SMD:L_0805_2012Metric, symbol Device:FerriteBead_Small
- J29: footprint (none) -> Connector_USB:USB_C_Receptacle_HRO_TYPE-C-31-M-12
- R10, R11: footprint (none) -> Resistor_SMD:R_0402_1005Metric
Connections:
- net VBUS: now also FB1.1
- new net: F1.1, FB1.2
- new net +5V: F1.2

Commit message: PCB
Parts:
- U5: MPN (none) -> 624-7693
- renumbered R10 to R30, R11 to R31
Changed lines of the file:
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@@
 		(dnp no)
 		(fields_autoplaced yes)
-		(property "Reference" "#PWR018"
+		(property "Reference" "#PWR0123"
 			(at 147.32 67.31 0)
 			(effects
@@
 			(project ""
 				(path "/61bc2d2d-cd10-4636-b1b1-3d875f78e40b/7a080ce4-c82c-46c4-8a5a-914178d680a1"
-					(reference "#PWR018")
+					(reference "#PWR0123")
 					(unit 1)
 				)
@@
 		(dnp no)
 		(fields_autoplaced yes)
-		(property "Reference" "#PWR093"
+		(property "Reference" "#PWR0121"
 			(at 124.46 91.44 0)
 			(effects
@@
 			(project ""
 				(path "/61bc2d2d-cd10-4636-b1b1-3d875f78e40b/7a080ce4-c82c-46c4-8a5a-914178d680a1"
-					(reference "#PWR093")
+					(reference "#PWR0121")
 					(unit 1)
 				)
@@
 		(dnp no)
 		(fields_autoplaced yes)
-		(property "Reference" "#PWR092"
+		(property "Reference" "#PWR0122"
 			(at 139.7 99.06 0)
 			(effects
@@
 			(project ""
 				(path "/61bc2d2d-cd10-4636-b1b1-3d875f78e40b/7a080ce4-c82c-46c4-8a5a-914178d680a1"
-					(reference "#PWR092")
+					(reference "#PWR0122")
 					(unit 1)
 				)
@@
 		(on_board yes)
 		(dnp no)
-		(property "Reference" "R11"
+		(property "Reference" "R31"
 			(at 119.126 87.122 90)
 			(effects
@@
 			(project ""
 				(path "/61bc2d2d-cd10-4636-b1b1-3d875f78e40b/7a080ce4-c82c-46c4-8a5a-914178d680a1"
-					(reference "R11")
+					(reference "R31")
 					(unit 1)
 				)
@@
 		(dnp no)
 		(fields_autoplaced yes)
-		(property "Reference" "#PWR091"
+		(property "Reference" "#PWR0120"
 			(at 86.36 121.92 0)
 			(effects
@@
 			(project ""
 				(path "/61bc2d2d-cd10-4636-b1b1-3d875f78e40b/7a080ce4-c82c-46c4-8a5a-914178d680a1"
-					(reference "#PWR091")
+					(reference "#PWR0120")
 					(unit 1)
 				)
@@
 		(dnp no)
 		(fields_autoplaced yes)
-		(property "Reference" "R10"
+		(property "Reference" "R30"
 			(at 119.38 77.47 90)
 			(effects
@@
 			(project ""
 				(path "/61bc2d2d-cd10-4636-b1b1-3d875f78e40b/7a080ce4-c82c-46c4-8a5a-914178d680a1"
-					(reference "R10")
+					(reference "R30")
 					(unit 1)
 				)
@@
 			(at 139.7 85.09 0)
 			(effects
+				(font
+					(size 1.27 1.27)
+				)
+				(hide yes)
+			)
+		)
+		(property "MPN" "624-7693"
+			(at 139.7 85.09 0)
+			(effects
