File: KiCAD/PCB projet ESE/Régulateurs.kicad_sch (KiCad schematic)
At the start: 0 parts

Commit message: finish first version of schematic
Parts:
- added BUxxSD1: ~, Régu:SSOP5_BUxxSD5, symbol Regulateur:BUxxSD5
- added C10A1, C1A1, C1A2, C27, C28, C2A1, C2A2, C33, C7A1: 22u, Capacitor_SMD:C_Elec_5x5.4, symbol Device:C_Small
- added C13, C19, C20, C21, C23, C24, C29, C30, C31: 0.1u, Capacitor_SMD:C_0402_1005Metric, symbol Device:C_Small
- added C16, C22: 1u, Capacitor_SMD:C_0603_1608Metric, symbol Device:C_Small
- added C25, C26, C32: 15p, Capacitor_SMD:C_0402_1005Metric, symbol Device:C_Small
- added L2, L3, L4: 4.7u, Inductor_SMD:L_0603_1608Metric, symbol Device:L_Small
- added MP3, MP4, MP5: ~, Régu:TSOT23-8, symbol Regulateur:MP1475
- added R12, R13, R14, R15, R24, R25: 100k, Resistor_SMD:R_0402_1005Metric, symbol Device:R_Small
- added R16, R17, R26: 20, Resistor_SMD:R_0402_1005Metric, symbol Device:R_Small
- added R18, R19: 16k, Resistor_SMD:R_0402_1005Metric, symbol Device:R_Small
- added R20: 7.68k, Resistor_SMD:R_0402_1005Metric, symbol Device:R_Small
- added R21: 4.9k, Resistor_SMD:R_0402_1005Metric, symbol Device:R_Small
- added R22, R23, R29: 40.2k, Resistor_SMD:R_0402_1005Metric, symbol Device:R_Small
- added R27: 33k, Resistor_SMD:R_0402_1005Metric, symbol Device:R_Small
- added R28: 16.3k, Resistor_SMD:R_0402_1005Metric, symbol Device:R_Small
Connections:
- new net: C26.1, R19.1, R21.1, R23.1
- new net: C19.1, MP3. (FB), R15.1
- new net: C32.1, R27.1, R28.1, R29.1
- new net: C23.1, R16.2
- new net: C23.2, L2.1, MP4. (FB)
- new net: C25.1, R18.1, R20.1, R22.1
- new net: C13.1, MP4. (FB), R14.1
- new net: MP5. (FB), R27.2
- new net: MP3. (FB), R19.2
- new net: MP3. (FB), R17.1
- new net: C24.2, L3.1, MP3. (FB)
- new net: C29.1, MP5. (FB), R25.1
- new net: MP4. (FB), R18.2
- new net: C24.1, R17.2
- new net: MP4. (FB), R16.1
- new net: C31.2, L4.1, MP5. (FB)
- new net: MP5. (FB), R26.1
- new net: C31.1, R26.2
- new net +14.8V: C1A1.2, C1A2.2, C20.2, C21.2, C30.2, C7A1.2, MP3. (FB), MP4. (FB), MP5. (FB), R12.1, R13.1, R24.1
- new net +2.8V: C10A1.2, C32.2, C33.2, L4.2, R29.2
- new net +3.3V: BUxxSD1. (NC), C22.1
- new net +5V: BUxxSD1. (NC), C16.1, C25.2, C27.2, C2A1.2, L2.2, R22.2
- new net +7.5V: C26.2, C28.2, C2A2.2, L3.2, R23.2
- new net EN/SYNC_2.8: MP5. (FB), R24.2
- new net EN/SYNC_5: MP4. (FB), R12.2
- new net EN/SYNC_7.5: MP3. (FB), R13.2
- new net GND: BUxxSD1. (NC), C10A1.1, C13.2, C16.2, C19.2, C1A1.1, C1A2.1, C20.1, C21.1, C22.2, C27.1, C28.1, C29.2, C2A1.1, C2A2.1, C30.1, C33.1, C7A1.1, MP3. (FB), MP4. (FB), MP5. (FB), R20.2, R21.2, R28.2
- new net PG_2.8: MP5. (FB), R25.2
- new net PG_5: MP4. (FB), R14.2
- new net PG_7.5: MP3. (FB), R15.2
- new net STBY_IN: BUxxSD1. (NC)
Other:
- note added: "2.8V/3A"
- note added: "5V/3A"
- note added: "7.5V/3A"
- note added: "Les LABELS (IN, VCC...) ne sont pas forcément exact, il faut les vérifier"
- note added: "Régulateur 2.8V/3A"
- note added: "Régulateur 3.3V"
- note added: "Régulateur 5V/3A"
- note added: "Régulateur 7.5V/3A à vérifier"

Commit message: PCB
Parts:
- removed MP3, MP4: ~, Régu:TSOT23-8, symbol Regulateur:MP1475
- added MP1, MP2: ~, Régu:TSOT23-8, symbol Regulateur:MP1475
- BUxxSD1: MPN (none) -> BU33SD5WG-TR
- MP3: renamed from MP5; MPN (none) -> MP1475DJ-LF-P
- renumbered C16 to C18, C1A1 to C19, C1A2 to C20, C13 to C21, C19 to C22, C20 to C23, C21 to C24, C22 to C25, C23 to C26, C24 to C27, C25 to C28, C26 to C29, C2A1 to C30, C2A2 to C31, C27 to C32, C28 to C33, C7A1 to C34, C29 to C35, C30 to C36, C31 to C37, C32 to C38, C10A1 to C39, C33 to C40
Connections:
- net +14.8V: now also MP3.2 (IN), MP1.2 (IN), MP2.2 (IN); no longer MP3. (FB)
- net +3.3V: now also BUxxSD1.5 (Vout); no longer BUxxSD1. (NC)
- net +5V: now also BUxxSD1.1 (Vin); no longer BUxxSD1. (NC)
- net EN/SYNC_2.8: now also MP3.6 (EN/SYNC); no longer MP3. (FB)
- net EN/SYNC_5: now also MP1.6 (EN/SYNC)
- net EN/SYNC_7.5: now also MP2.6 (EN/SYNC)
- net GND: now also BUxxSD1.2 (GND), MP3.4 (GND), MP1.4 (GND), MP2.4 (GND); no longer BUxxSD1. (NC), MP3. (FB)
- net PG_2.8: now also MP3.1 (PG); no longer MP3. (FB)
- net PG_5: now also MP1.1 (PG)
- net PG_7.5: now also MP2.1 (PG)
- net at C22.1, R15.1: now also MP2.7 (VCC)
- net at C26.2, L2.1: now also MP1.3 (SW)
- net at C21.1, R14.1: now also MP1.7 (VCC)
- net at R27.2: now also MP3.8 (FB); no longer MP3. (FB)
- net at R19.2: now also MP2.8 (FB)
- net at R17.1: now also MP2.5 (BST)
- net at C27.2, L3.1: now also MP2.3 (SW)
- net at C35.1, R25.1: now also MP3.7 (VCC); no longer MP3. (FB)
- net at R18.2: now also MP1.8 (FB)
- net at R16.1: now also MP1.5 (BST)
- net at C37.2, L4.1: now also MP3.3 (SW); no longer MP3. (FB)
- net at R26.1: now also MP3.5 (BST); no longer MP3. (FB)
