File: KiCAD/PCB projet ESE/TOF.kicad_sch (KiCad schematic)
At the start: 10 parts, among them J1 Conn_01x06, J10 Conn_01x06, J11 Conn_01x06, J2 Conn_01x06, J3 Conn_01x06, J4 Conn_01x06, J7 Conn_01x06, J8 Conn_01x06

Commit message: finish first version of schematic
Parts:
- J1, J10, J11, J2, J3, J4, J7, J8: footprint (none) -> Connector_JST:JST_PH_B6B-PH-K_1x06_P2.00mm_Vertical
- R3, R4: footprint (none) -> Resistor_SMD:R_0402_1005Metric
Changed lines of the file:
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@@
 			)
 		)
-		(property "Footprint" ""
+		(property "Footprint" "Connector_JST:JST_PH_B6B-PH-K_1x06_P2.00mm_Vertical"
 			(at 92.71 90.17 0)
 			(effects
@@
 			)
 		)
-		(property "Footprint" ""
+		(property "Footprint" "Connector_JST:JST_PH_B6B-PH-K_1x06_P2.00mm_Vertical"
 			(at 111.76 114.3 0)
 			(effects
@@
 			)
 		)
-		(property "Footprint" ""
+		(property "Footprint" "Connector_JST:JST_PH_B6B-PH-K_1x06_P2.00mm_Vertical"
 			(at 130.81 90.17 0)
 			(effects
@@
 			)
 		)
-		(property "Footprint" ""
+		(property "Footprint" "Resistor_SMD:R_0402_1005Metric"
 			(at 140.97 111.76 0)
 			(effects
@@
 			)
 		)
-		(property "Footprint" ""
+		(property "Footprint" "Connector_JST:JST_PH_B6B-PH-K_1x06_P2.00mm_Vertical"
 			(at 92.71 67.31 0)
 			(effects
@@
 			)
 		)
-		(property "Footprint" ""
+		(property "Footprint" "Connector_JST:JST_PH_B6B-PH-K_1x06_P2.00mm_Vertical"
 			(at 111.76 67.31 0)
 			(effects
@@
 			)
 		)
-		(property "Footprint" ""
+		(property "Footprint" "Connector_JST:JST_PH_B6B-PH-K_1x06_P2.00mm_Vertical"
 			(at 92.71 114.3 0)
 			(effects
@@
 			)
 		)
-		(property "Footprint" ""
+		(property "Footprint" "Connector_JST:JST_PH_B6B-PH-K_1x06_P2.00mm_Vertical"
 			(at 111.76 90.17 0)
 			(effects
@@
 			)
 		)
-		(property "Footprint" ""
+		(property "Footprint" "Connector_JST:JST_PH_B6B-PH-K_1x06_P2.00mm_Vertical"
 			(at 130.81 67.31 0)
 			(effects
@@
 			)
 		)
-		(property "Footprint" ""
+		(property "Footprint" "Resistor_SMD:R_0402_1005Metric"
 			(at 134.62 111.76 0)
 			(effects

Commit message: PCB
Parts:
- renumbered J7 to J10, J2 to J11, J4 to J12, J8 to J13, J10 to J14, J11 to J15, J1 to J8, J3 to J9, R3 to R10, R4 to R11
Changed lines of the file:
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@@
 		(on_board yes)
 		(dnp no)
-		(property "Reference" "J3"
+		(property "Reference" "J9"
 			(at 92.71 76.2 0)
 			(effects
@@
 			(project "PCB projet ESE"
 				(path "/61bc2d2d-cd10-4636-b1b1-3d875f78e40b/261d7bb0-1163-45ca-901d-11d0cf203b6b"
-					(reference "J3")
+					(reference "J9")
 					(unit 1)
 				)
@@
 		(dnp no)
 		(fields_autoplaced yes)
-		(property "Reference" "#PWR070"
+		(property "Reference" "#PWR067"
 			(at 140.97 107.95 0)
 			(effects
@@
 			(project "PCB projet ESE"
 				(path "/61bc2d2d-cd10-4636-b1b1-3d875f78e40b/261d7bb0-1163-45ca-901d-11d0cf203b6b"
-					(reference "#PWR070")
+					(reference "#PWR067")
 					(unit 1)
 				)
@@
 		(dnp no)
 		(fields_autoplaced yes)
-		(property "Reference" "#PWR049"
+		(property "Reference" "#PWR058"
 			(at 123.19 106.68 0)
 			(effects
@@
 			(project "PCB projet ESE"
 				(path "/61bc2d2d-cd10-4636-b1b1-3d875f78e40b/261d7bb0-1163-45ca-901d-11d0cf203b6b"
-					(reference "#PWR049")
+					(reference "#PWR058")
 					(unit 1)
 				)
@@
 		(dnp no)
 		(fields_autoplaced yes)
-		(property "Reference" "#PWR042"
+		(property "Reference" "#PWR059"
 			(at 120.65 66.04 0)
 			(effects
@@
 			(project "PCB projet ESE"
 				(path "/61bc2d2d-cd10-4636-b1b1-3d875f78e40b/261d7bb0-1163-45ca-901d-11d0cf203b6b"
-					(reference "#PWR042")
+					(reference "#PWR059")
 					(unit 1)
 				)
@@
 		(dnp no)
 		(fields_autoplaced yes)
-		(property "Reference" "#PWR054"
+		(property "Reference" "#PWR066"
 			(at 139.7 88.9 0)
 			(effects
@@
 			(project "PCB projet ESE"
 				(path "/61bc2d2d-cd10-4636-b1b1-3d875f78e40b/261d7bb0-1163-45ca-901d-11d0cf203b6b"
-					(reference "#PWR054")
+					(reference "#PWR066")
 					(unit 1)
 				)
@@
 		(on_board yes)
 		(dnp no)
-		(property "Reference" "J8"
+		(property "Reference" "J13"
 			(at 111.76 100.33 0)
 			(effects
@@
 			(project "PCB projet ESE"
 				(path "/61bc2d2d-cd10-4636-b1b1-3d875f78e40b/261d7bb0-1163-45ca-901d-11d0cf203b6b"
-					(reference "J8")
+					(reference "J13")
 					(unit 1)
 				)
@@
 		(on_board yes)
 		(dnp no)
-		(property "Reference" "J11"
+		(property "Reference" "J15"
 			(at 130.81 76.2 0)
 			(effects
@@
 			(project "PCB projet ESE"
 				(path "/61bc2d2d-cd10-4636-b1b1-3d875f78e40b/261d7bb0-1163-45ca-901d-11d0cf203b6b"
-					(reference "J11")
+					(reference "J15")
 					(unit 1)
 				)
@@
 		(dnp no)
 		(fields_autoplaced yes)
-		(property "Reference" "#PWR040"
+		(property "Reference" "#PWR050"
 			(at 104.14 59.69 0)
 			(effects
@@
 			(project "PCB projet ESE"
 				(path "/61bc2d2d-cd10-4636-b1b1-3d875f78e40b/261d7bb0-1163-45ca-901d-11d0cf203b6b"
-					(reference "#PWR040")
+					(reference "#PWR050")
 					(unit 1)
 				)
@@
 		(dnp no)
 		(fields_autoplaced yes)
-		(property "Reference" "R4"
+		(property "Reference" "R11"
 			(at 143.51 110.4899 0)
 			(effects
@@
 			(project "PCB projet ESE"
 				(path "/61bc2d2d-cd10-4636-b1b1-3d875f78e40b/261d7bb0-1163-45ca-901d-11d0cf203b6b"
-					(reference "R4")
+					(reference "R11")
 					(unit 1)
 				)
@@
 		(on_board yes)
 		(dnp no)
-		(property "Reference" "J1"
+		(property "Reference" "J8"
 			(at 92.71 53.34 0)
 			(effects
@@
 			(project "PCB projet ESE"
 				(path "/61bc2d2d-cd10-4636-b1b1-3d875f78e40b/261d7bb0-1163-45ca-901d-11d0cf203b6b"
-					(reference "J1")
+					(reference "J8")
 					(unit 1)
 				)
@@
 		(dnp no)
 		(fields_autoplaced yes)
-		(property "Reference" "#PWR039"
+		(property "Reference" "#PWR053"
 			(at 101.6 66.04 0)
 			(effects
@@
 			(project "PCB projet ESE"
 				(path "/61bc2d2d-cd10-4636-b1b1-3d875f78e40b/261d7bb0-1163-45ca-901d-11d0cf203b6b"
-					(reference "#PWR039")
+					(reference "#PWR053")
 					(unit 1)
 				)
@@
 		(dnp no)
 		(fields_autoplaced yes)
-		(property "Reference" "#PWR046"
+		(property "Reference" "#PWR060"
 			(at 120.65 88.9 0)
 			(effects
@@
 			(project "PCB projet ESE"
 				(path "/61bc2d2d-cd10-4636-b1b1-3d875f78e40b/261d7bb0-1163-45ca-901d-11d0cf203b6b"
-					(reference "#PWR046")
+					(reference "#PWR060")
 					(unit 1)
 				)
@@
 		(dnp no)
 		(fields_autoplaced yes)
-		(property "Reference" "#PWR047"
+		(property "Reference" "#PWR052"
 			(at 104.14 106.68 0)
 			(effects
@@
 			(project "PCB projet ESE"
 				(path "/61bc2d2d-cd10-4636-b1b1-3d875f78e40b/261d7bb0-1163-45ca-901d-11d0cf203b6b"
-					(reference "#PWR047")
+					(reference "#PWR052")
 					(unit 1)
 				)
@@
 		(dnp no)
 		(fields_autoplaced yes)
-		(property "Reference" "#PWR053"
+		(property "Reference" "#PWR065"
 			(at 139.7 66.04 0)
 			(effects
@@
 			(project "PCB projet ESE"
 				(path "/61bc2d2d-cd10-4636-b1b1-3d875f78e40b/261d7bb0-1163-45ca-901d-11d0cf203b6b"
-					(reference "#PWR053")
+					(reference "#PWR065")
 					(unit 1)
 				)
@@
 		(on_board yes)
 		(dnp no)
-		(property "Reference" "J2"
+		(property "Reference" "J11"
 			(at 111.76 53.34 0)
 			(effects
@@
 			(project "PCB projet ESE"
 				(path "/61bc2d2d-cd10-4636-b1b1-3d875f78e40b/261d7bb0-1163-45ca-901d-11d0cf203b6b"
-					(reference "J2")
+					(reference "J11")
 					(unit 1)
 				)
@@
 		(dnp no)
 		(fields_autoplaced yes)
-		(property "Reference" "#PWR069"
+		(property "Reference" "#PWR062"
 			(at 134.62 107.95 0)
 			(effects
@@
 			(project "PCB projet ESE"
 				(path "/61bc2d2d-cd10-4636-b1b1-3d875f78e40b/261d7bb0-1163-45ca-901d-11d0cf203b6b"
-					(reference "#PWR069")
+					(reference "#PWR062")
 					(unit 1)
 				)
@@
 		(on_board yes)
 		(dnp no)
-		(property "Reference" "J7"
+		(property "Reference" "J10"
 			(at 92.71 100.33 0)
 			(effects
@@
 			(project "PCB projet ESE"
 				(path "/61bc2d2d-cd10-4636-b1b1-3d875f78e40b/261d7bb0-1163-45ca-901d-11d0cf203b6b"
-					(reference "J7")
+					(reference "J10")
 					(unit 1)
 				)
@@
 		(dnp no)
 		(fields_autoplaced yes)
-		(property "Reference" "#PWR041"
+		(property "Reference" "#PWR056"
 			(at 123.19 59.69 0)
 			(effects
@@
 			(project "PCB projet ESE"
 				(path "/61bc2d2d-cd10-4636-b1b1-3d875f78e40b/261d7bb0-1163-45ca-901d-11d0cf203b6b"
-					(reference "#PWR041")
+					(reference "#PWR056")
 					(unit 1)
 				)
@@
 		(dnp no)
 		(fields_autoplaced yes)
-		(property "Reference" "#PWR048"
+		(property "Reference" "#PWR055"
 			(at 101.6 113.03 0)
 			(effects
@@
 			(project "PCB projet ESE"
 				(path "/61bc2d2d-cd10-4636-b1b1-3d875f78e40b/261d7bb0-1163-45ca-901d-11d0cf203b6b"
-					(reference "#PWR048")
+					(reference "#PWR055")
 					(unit 1)
 				)
@@
 		(dnp no)
 		(fields_autoplaced yes)
-		(property "Reference" "#PWR043"
+		(property "Reference" "#PWR051"
 			(at 104.14 82.55 0)
 			(effects
@@
 			(project "PCB projet ESE"
 				(path "/61bc2d2d-cd10-4636-b1b1-3d875f78e40b/261d7bb0-1163-45ca-901d-11d0cf203b6b"
-					(reference "#PWR043")
+					(reference "#PWR051")
 					(unit 1)
 				)
@@
 		(dnp no)
 		(fields_autoplaced yes)
-		(property "Reference" "#PWR045"
+		(property "Reference" "#PWR057"
 			(at 123.19 82.55 0)
 			(effects
@@
 			(project "PCB projet ESE"
 				(path "/61bc2d2d-cd10-4636-b1b1-3d875f78e40b/261d7bb0-1163-45ca-901d-11d0cf203b6b"
-					(reference "#PWR045")
+					(reference "#PWR057")
 					(unit 1)
 				)
@@
 		(dnp no)
 		(fields_autoplaced yes)
-		(property "Reference" "#PWR050"
+		(property "Reference" "#PWR061"
 			(at 120.65 113.03 0)
 			(effects
@@
 			(project "PCB projet ESE"
 				(path "/61bc2d2d-cd10-4636-b1b1-3d875f78e40b/261d7bb0-1163-45ca-901d-11d0cf203b6b"
-					(reference "#PWR050")
+					(reference "#PWR061")
 					(unit 1)
 				)
@@
 		(on_board yes)
 		(dnp no)
-		(property "Reference" "J4"
+		(property "Reference" "J12"
 			(at 111.76 76.2 0)
 			(effects
@@
 			(project "PCB projet ESE"
 				(path "/61bc2d2d-cd10-4636-b1b1-3d875f78e40b/261d7bb0-1163-45ca-901d-11d0cf203b6b"
-					(reference "J4")
+					(reference "J12")
 					(unit 1)
 				)
@@
 		(on_board yes)
 		(dnp no)
-		(property "Reference" "J10"
+		(property "Reference" "J14"
 			(at 130.81 53.34 0)
 			(effects
@@
 			(project "PCB projet ESE"
 				(path "/61bc2d2d-cd10-4636-b1b1-3d875f78e40b/261d7bb0-1163-45ca-901d-11d0cf203b6b"
-					(reference "J10")
+					(reference "J14")
 					(unit 1)
 				)
@@
 		(dnp no)
 		(fields_autoplaced yes)
-		(property "Reference" "R3"
+		(property "Reference" "R10"
 			(at 137.16 110.4899 0)
 			(effects
@@
 			(project "PCB projet ESE"
 				(path "/61bc2d2d-cd10-4636-b1b1-3d875f78e40b/261d7bb0-1163-45ca-901d-11d0cf203b6b"
-					(reference "R3")
+					(reference "R10")
 					(unit 1)
 				)
@@
 		(dnp no)
 		(fields_autoplaced yes)
-		(property "Reference" "#PWR052"
+		(property "Reference" "#PWR064"
 			(at 142.24 82.55 0)
 			(effects
@@
 			(project "PCB projet ESE"
 				(path "/61bc2d2d-cd10-4636-b1b1-3d875f78e40b/261d7bb0-1163-45ca-901d-11d0cf203b6b"
-					(reference "#PWR052")
+					(reference "#PWR064")
 					(unit 1)
 				)
@@
 		(dnp no)
 		(fields_autoplaced yes)
-		(property "Reference" "#PWR051"
+		(property "Reference" "#PWR063"
 			(at 142.24 59.69 0)
 			(effects
@@
 			(project "PCB projet ESE"
 				(path "/61bc2d2d-cd10-4636-b1b1-3d875f78e40b/261d7bb0-1163-45ca-901d-11d0cf203b6b"
-					(reference "#PWR051")
+					(reference "#PWR063")
 					(unit 1)
 				)
@@
 		(dnp no)
 		(fields_autoplaced yes)
-		(property "Reference" "#PWR044"
+		(property "Reference" "#PWR054"
 			(at 101.6 88.9 0)
 			(effects
@@
 			(project "PCB projet ESE"
 				(path "/61bc2d2d-cd10-4636-b1b1-3d875f78e40b/261d7bb0-1163-45ca-901d-11d0cf203b6b"
-					(reference "#PWR044")
-					(unit 1)
-				)
+					(reference "#PWR054")
+					(unit 1)
+				)
