File: KiCAD/PCB projet ESE/neopixel.kicad_sch (KiCad schematic)
At the start: 5 parts, among them J14 Conn_01x03, J17 Conn_01x03, J18 Conn_01x03, J19 Conn_01x03, J20 Conn_01x03

Commit message: finish first version of schematic
Parts:
- J14, J17, J18, J19, J20: footprint (none) -> Connector_JST:JST_PH_B3B-PH-K_1x03_P2.00mm_Vertical
Changed lines of the file:
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@@
 			)
 		)
-		(property "Footprint" ""
+		(property "Footprint" "Connector_JST:JST_PH_B3B-PH-K_1x03_P2.00mm_Vertical"
 			(at 95.25 101.6 0)
 			(effects
@@
 			)
 		)
-		(property "Footprint" ""
+		(property "Footprint" "Connector_JST:JST_PH_B3B-PH-K_1x03_P2.00mm_Vertical"
 			(at 106.68 74.93 0)
 			(effects
@@
 			)
 		)
-		(property "Footprint" ""
+		(property "Footprint" "Connector_JST:JST_PH_B3B-PH-K_1x03_P2.00mm_Vertical"
 			(at 82.55 73.66 0)
 			(effects
@@
 			)
 		)
-		(property "Footprint" ""
+		(property "Footprint" "Connector_JST:JST_PH_B3B-PH-K_1x03_P2.00mm_Vertical"
 			(at 134.62 76.2 0)
 			(effects
@@
 			)
 		)
-		(property "Footprint" ""
+		(property "Footprint" "Connector_JST:JST_PH_B3B-PH-K_1x03_P2.00mm_Vertical"
 			(at 125.73 101.6 0)
 			(effects

Commit message: PCB
Parts:
- renumbered J14 to J16, J19 to J17, J17 to J18, J20 to J19, J18 to J20
Changed lines of the file:
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@@
 		(dnp no)
 		(fields_autoplaced yes)
-		(property "Reference" "#PWR071"
+		(property "Reference" "#PWR072"
 			(at 111.76 83.82 0)
 			(effects
@@
 			(project "PCB projet ESE"
 				(path "/61bc2d2d-cd10-4636-b1b1-3d875f78e40b/ea158019-ab8a-47c5-8451-862ac372ee0d"
-					(reference "#PWR071")
+					(reference "#PWR072")
 					(unit 1)
 				)
@@
 		(dnp no)
 		(fields_autoplaced yes)
-		(property "Reference" "#PWR057"
+		(property "Reference" "#PWR068"
 			(at 87.63 82.55 0)
 			(effects
@@
 			(project "PCB projet ESE"
 				(path "/61bc2d2d-cd10-4636-b1b1-3d875f78e40b/ea158019-ab8a-47c5-8451-862ac372ee0d"
-					(reference "#PWR057")
+					(reference "#PWR068")
 					(unit 1)
 				)
@@
 		(dnp no)
 		(fields_autoplaced yes)
-		(property "Reference" "J19"
+		(property "Reference" "J17"
 			(at 95.25 92.71 0)
 			(effects
@@
 			(project "PCB projet ESE"
 				(path "/61bc2d2d-cd10-4636-b1b1-3d875f78e40b/ea158019-ab8a-47c5-8451-862ac372ee0d"
-					(reference "J19")
+					(reference "J17")
 					(unit 1)
 				)
@@
 		(dnp no)
 		(fields_autoplaced yes)
-		(property "Reference" "#PWR072"
+		(property "Reference" "#PWR073"
 			(at 118.11 76.2 0)
 			(effects
@@
 			(project "PCB projet ESE"
 				(path "/61bc2d2d-cd10-4636-b1b1-3d875f78e40b/ea158019-ab8a-47c5-8451-862ac372ee0d"
-					(reference "#PWR072")
+					(reference "#PWR073")
 					(unit 1)
 				)
@@
 		(dnp no)
 		(fields_autoplaced yes)
-		(property "Reference" "#PWR077"
+		(property "Reference" "#PWR074"
 			(at 130.81 110.49 0)
 			(effects
@@
 			(project "PCB projet ESE"
 				(path "/61bc2d2d-cd10-4636-b1b1-3d875f78e40b/ea158019-ab8a-47c5-8451-862ac372ee0d"
-					(reference "#PWR077")
+					(reference "#PWR074")
 					(unit 1)
 				)
@@
 		(dnp no)
 		(fields_autoplaced yes)
-		(property "Reference" "J17"
+		(property "Reference" "J18"
 			(at 106.68 66.04 0)
 			(effects
@@
 			(project "PCB projet ESE"
 				(path "/61bc2d2d-cd10-4636-b1b1-3d875f78e40b/ea158019-ab8a-47c5-8451-862ac372ee0d"
-					(reference "J17")
+					(reference "J18")
 					(unit 1)
 				)
@@
 		(dnp no)
 		(fields_autoplaced yes)
-		(property "Reference" "#PWR074"
+		(property "Reference" "#PWR077"
 			(at 146.05 77.47 0)
 			(effects
@@
 			(project "PCB projet ESE"
 				(path "/61bc2d2d-cd10-4636-b1b1-3d875f78e40b/ea158019-ab8a-47c5-8451-862ac372ee0d"
-					(reference "#PWR074")
+					(reference "#PWR077")
 					(unit 1)
 				)
@@
 		(dnp no)
 		(fields_autoplaced yes)
-		(property "Reference" "#PWR058"
+		(property "Reference" "#PWR069"
 			(at 93.98 74.93 0)
 			(effects
@@
 			(project "PCB projet ESE"
 				(path "/61bc2d2d-cd10-4636-b1b1-3d875f78e40b/ea158019-ab8a-47c5-8451-862ac372ee0d"
-					(reference "#PWR058")
+					(reference "#PWR069")
 					(unit 1)
 				)
@@
 		(dnp no)
 		(fields_autoplaced yes)
-		(property "Reference" "#PWR076"
+		(property "Reference" "#PWR071"
 			(at 106.68 102.87 0)
 			(effects
@@
 			(project "PCB projet ESE"
 				(path "/61bc2d2d-cd10-4636-b1b1-3d875f78e40b/ea158019-ab8a-47c5-8451-862ac372ee0d"
-					(reference "#PWR076")
+					(reference "#PWR071")
 					(unit 1)
 				)
@@
 		(dnp no)
 		(fields_autoplaced yes)
-		(property "Reference" "J14"
+		(property "Reference" "J16"
 			(at 82.55 64.77 0)
 			(effects
@@
 			(project "PCB projet ESE"
 				(path "/61bc2d2d-cd10-4636-b1b1-3d875f78e40b/ea158019-ab8a-47c5-8451-862ac372ee0d"
-					(reference "J14")
+					(reference "J16")
 					(unit 1)
 				)
@@
 		(dnp no)
 		(fields_autoplaced yes)
-		(property "Reference" "J18"
+		(property "Reference" "J20"
 			(at 134.62 67.31 0)
 			(effects
@@
 			(project "PCB projet ESE"
 				(path "/61bc2d2d-cd10-4636-b1b1-3d875f78e40b/ea158019-ab8a-47c5-8451-862ac372ee0d"
-					(reference "J18")
+					(reference "J20")
 					(unit 1)
 				)
@@
 		(dnp no)
 		(fields_autoplaced yes)
-		(property "Reference" "#PWR075"
+		(property "Reference" "#PWR070"
 			(at 100.33 110.49 0)
 			(effects
@@
 			(project "PCB projet ESE"
 				(path "/61bc2d2d-cd10-4636-b1b1-3d875f78e40b/ea158019-ab8a-47c5-8451-862ac372ee0d"
-					(reference "#PWR075")
+					(reference "#PWR070")
 					(unit 1)
 				)
@@
 		(dnp no)
 		(fields_autoplaced yes)
-		(property "Reference" "#PWR078"
+		(property "Reference" "#PWR075"
 			(at 137.16 102.87 0)
 			(effects
@@
 			(project "PCB projet ESE"
 				(path "/61bc2d2d-cd10-4636-b1b1-3d875f78e40b/ea158019-ab8a-47c5-8451-862ac372ee0d"
-					(reference "#PWR078")
+					(reference "#PWR075")
 					(unit 1)
 				)
@@
 		(dnp no)
 		(fields_autoplaced yes)
-		(property "Reference" "J20"
+		(property "Reference" "J19"
 			(at 125.73 92.71 0)
 			(effects
@@
 			(project "PCB projet ESE"
 				(path "/61bc2d2d-cd10-4636-b1b1-3d875f78e40b/ea158019-ab8a-47c5-8451-862ac372ee0d"
-					(reference "J20")
+					(reference "J19")
 					(unit 1)
 				)
@@
 		(dnp no)
 		(fields_autoplaced yes)
-		(property "Reference" "#PWR073"
+		(property "Reference" "#PWR076"
 			(at 139.7 85.09 0)
 			(effects
@@
 			(project "PCB projet ESE"
 				(path "/61bc2d2d-cd10-4636-b1b1-3d875f78e40b/ea158019-ab8a-47c5-8451-862ac372ee0d"
-					(reference "#PWR073")
-					(unit 1)
-				)
+					(reference "#PWR076")
+					(unit 1)
+				)
