File: KiCAD/PCB projet ESE/PCB projet ESE.kicad_sch (KiCad schematic)
At the start: 18 parts, among them U1 STM32WB55CEUx, U2 ADXL343, U3 ZXBM5210-SP, Y1 32M

Commit message: maj schematic
Parts:
- added C14, C16, C17: 100n, symbol Device:C_Small
- added C15, C18: 4.7u, symbol Device:C_Small
- added D1, D2, D3, D4, D5: LED, symbol Device:LED
- added H1, H2, H3, H4: MountingHole_Pad, symbol Mechanical:MountingHole_Pad
- added J1, J10, J11, J16, J2, J3, J4, J5, J6, J7, J8: Conn_01x06, symbol Connector_Generic:Conn_01x06
- added J12, J15: Conn_01x04, symbol Connector_Generic:Conn_01x04
- added J13: Conn_01x02, symbol Connector_Generic:Conn_01x02
- added J14: Conn_01x03, symbol Connector_Generic:Conn_01x03
- added J9: Conn_ST_STDC14, symbol Connector:Conn_ST_STDC14
- added R1, R2, R3, R4: 1k, symbol Device:R_Small
- added R5: 6k55, symbol Device:R_Small
- added R6: 2k9, symbol Device:R_Small
- added R7: 1k65, symbol Device:R_Small
- added R8: 800, symbol Device:R_Small
- added R9: 550, symbol Device:R_Small
- added SW1: SW_SPST, symbol Switch:SW_SPST
- added SW2: SW_SPDT, symbol Switch:SW_SPDT
- added U4: ZXBM5210-SP, Package_SO:Diodes_SO-8EP, symbol Driver_Motor:ZXBM5210-SP
- added U5: ~, symbol ESE:MP1475
Connections:
- net +3.3V: now also J12.1 (Pin_1), J5.5 (Pin_5), J6.5 (Pin_5), J9.3 (VCC), R1.1, R2.1, R3.1, R4.1, R8.1
- net GND: now also U2.12 (SDO/ADDR), U3.8 (GND), U3.9 (GND), C14.2, C15.1, C16.2, C17.2, C18.1, D1.1 (K), D2.1 (K), D3.1 (K), D4.1 (K), D5.1 (K), H1.1, H2.1, H3.1, H4.1, J1.6 (Pin_6), J10.6 (Pin_6), J11.6 (Pin_6), J12.2 (Pin_2), J13.1 (Pin_1), J14.1 (Pin_1), J15.4 (Pin_4), J16.3 (Pin_3), J2.6 (Pin_6), J3.6 (Pin_6), J4.6 (Pin_6), J5.1 (Pin_1), J5.2 (Pin_2), J6.1 (Pin_1), J6.2 (Pin_2), J7.6 (Pin_6), J8.6 (Pin_6), J9.11 (GNDDetect), J9.5 (GND), J9.7 (GND), SW1.2 (B), U4.8 (GND), U4.9 (GND)
- net NRST: now reaches U1.7 (NRST)
- net NRST: now also C16.1, J9.12 (~{RST}), SW1.1 (A)
- net Encodeur phase A 1: now reaches U3.1 (OUT1)
- net Encodeur phase A 1: now also J5.3 (Pin_3)
- net at U3.2 (VM): now also C15.2
- net +7.5V: now reaches U3.3 (VDD)
- net +7.5V: now also U3.6 (VREF), C14.1, C17.1, J5.6 (Pin_6), J6.6 (Pin_6), R6.1, U4.3 (VDD), U4.6 (VREF)
- net PWM FWD 1: now reaches U3.4 (FWD)
- net PWM REV 1: now reaches U3.5 (REV)
- net Encodeur Phase B 1: now reaches U3.7 (OUT2)
- net Encodeur Phase B 1: now also J5.4 (Pin_4)
- net Accel SDA: now reaches U2.13 (SDA/SDI/SDIO)
- net Accel SDA: now also R1.2
- net Accel SCL: now reaches U2.14 (SCL/SCLK)
- net Accel SCL: now also R2.2
- net INT 1: now reaches U2.8 (INT1)
- net INT 2: now reaches U2.9 (INT2)
- new net: C18.2, U4.2 (VM)
- new net: D1.2 (A), R9.2
- new net: D4.2 (A), R7.2
- new net: D5.2 (A), R5.2
- new net: J13.2 (Pin_2), SW2.2 (B)
- new net: D2.2 (A), R8.2
- new net: D3.2 (A), R6.2
- new net +14.8V: R5.1, SW2.1 (A)
- new net +2.8V: J1.5 (Pin_5), J10.5 (Pin_5), J11.5 (Pin_5), J2.5 (Pin_5), J3.5 (Pin_5), J4.5 (Pin_5), J7.5 (Pin_5), J8.5 (Pin_5), R9.1
- new net +5V: J12.4 (Pin_4), J14.3 (Pin_3), J15.3 (Pin_3), J16.2 (Pin_2), R7.1
- new net Encodeur Phase B 2: J6.4 (Pin_4), U4.7 (OUT2)
- new net Encodeur phase A 2: J6.3 (Pin_3), U4.1 (OUT1)
- new net INT: J1.1 (Pin_1), J10.1 (Pin_1), J11.1 (Pin_1), J2.1 (Pin_1), J3.1 (Pin_1), J4.1 (Pin_1), J7.1 (Pin_1), J8.1 (Pin_1)
- new net Lidar Output : J12.3 (Pin_3)
- new net PWM FWD 2: U4.4 (FWD)
- new net PWM REV 2: U4.5 (REV)
- new net PWM_LED: J14.2 (Pin_2)
- new net SCL TOF: J1.2 (Pin_2), J10.2 (Pin_2), J11.2 (Pin_2), J2.2 (Pin_2), J3.2 (Pin_2), J4.2 (Pin_2), J7.2 (Pin_2), J8.2 (Pin_2)
- new net SDA TOF: J1.4 (Pin_4), J10.4 (Pin_4), J11.4 (Pin_4), J2.4 (Pin_4), J3.4 (Pin_4), J4.4 (Pin_4), J7.4 (Pin_4), J8.4 (Pin_4), R3.2, R4.2
- new net SWCLK: J9.6 (JCLK/SWCLK)
- new net SWDIO: J9.4 (JTMS/SWDIO)
- new net UART_Debug_RX: J9.13 (VCP_RX)
- new net UART_Debug_TX: J9.14 (VCP_TX)
- new net UART_HC05_RX: J16.5 (Pin_5)
- new net UART_HC05_TX: J16.4 (Pin_4)
- new net UART_mp3_RX: J15.1 (Pin_1)
- new net UART_mp3_TX: J15.2 (Pin_2)
- new net XSHUT 1: J1.3 (Pin_3)
- new net XSHUT 2: J2.3 (Pin_3)
- new net XSHUT 3: J10.3 (Pin_3)
- new net XSHUT 4: J3.3 (Pin_3)
- new net XSHUT 5: J4.3 (Pin_3)
- new net XSHUT 6: J11.3 (Pin_3)
- new net XSHUT 7: J7.3 (Pin_3)
- new net XSHUT 8: J8.3 (Pin_3)
- no-connect marks 2 -> 8
Other:
- note added: "!!"
- note added: "Accéléromètre"
- note added: "Conn"
- note added: "I/O"
- note added: "Lidar"
- note added: "Moteurs"
- note added: "Régulateurs"
- note added: "TOF"
- note added: "Trous de fixation"
- note added: "USB C pour rasbpi 5V/3A (voir même 4A en pointe)"
- note removed: "can be connected to a GPIO"
- moved on the sheet: C1, C10, C11, C12, C13, C2, C3, C4, C5, C6, C7, C8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

Commit message: pcb schematic maj
Parts:
- removed C13: 100p, symbol Device:C_Small
- removed C16: 100n, symbol Device:C_Small
- removed J1, J10, J11, J2, J3, J4, J7, J8: Conn_01x06, symbol Connector_Generic:Conn_01x06
- removed J14: Conn_01x03, symbol Connector_Generic:Conn_01x03
- removed R3, R4: 1k, symbol Device:R_Small
- removed U1: STM32WB55CEUx, Package_DFN_QFN:QFN-48-1EP_7x7mm_P0.5mm_EP5.6x5.6mm, symbol MCU_ST_STM32WB:STM32WB55CEUx
- removed U5: ~, symbol ESE:MP1475
- removed Y1: 32M, symbol Device:Crystal_Small
- added U1: STM32G474RETx, Package_QFP:LQFP-64_10x10mm_P0.5mm, symbol MCU_ST_STM32G4:STM32G474RETx
- C1: value 10n -> 4u7
- C10, C6: value 4.7u -> 1u
- C2: value 1u -> 100n
- C9: value 4.7u -> 10n
- L1: value 10u -> 39n
Connections:
- net +3.3V: now also C9.1, L1.1, U1.1 (VBAT), U1.16 (VDD), U1.28 (VREF+), U1.29 (VDDA), U1.32 (VDD), U1.48 (VDD), U1.64 (VDD); no longer C12.1
- net GND: now also U1.15 (VSS), U1.27 (VSSA), U1.31 (VSS), U1.47 (VSS), U1.63 (VSS)
- net NRST: now also C12.1, U1.7 (PG10)
Other:
- added sheet LED NEOPIXEL (neopixel.kicad_sch)
- added sheet Rasbpi (Rasbpi.kicad_sch)
- added sheet Régulateurs (Régulateurs.kicad_sch)
- added sheet Servo FS90 (ServoFS90.kicad_sch)
- added sheet TOF (TOF.kicad_sch)
- note removed: "!!"
- note removed: "TOF"

Commit message: finish first version of schematic
Parts:
- added C34: 100n, Capacitor_SMD:C_0402_1005Metric, symbol Device:C_Small
- added R30: 47k, Resistor_SMD:R_0402_1005Metric, symbol Device:R_Small
- added R31: 10k, Resistor_SMD:R_0402_1005Metric, symbol Device:R_Small
- C1, C10, C15, C18, C6, C8: footprint (none) -> Capacitor_SMD:C_0603_1608Metric
- C11, C12, C14, C17, C2, C3, C4, C5, C7, C9: footprint (none) -> Capacitor_SMD:C_0402_1005Metric
- D1, D2, D3, D4, D5: footprint (none) -> LED_SMD:LED_0603_1608Metric
- H1, H2, H3, H4: footprint (none) -> MountingHole:MountingHole_3.2mm_M3_Pad_Via
- J12, J15: footprint (none) -> Connector_JST:JST_PH_B4B-PH-K_1x04_P2.00mm_Vertical
- J13: footprint (none) -> Connector_AMASS:AMASS_XT60-M_1x02_P7.20mm_Vertical
- J16, J5, J6: footprint (none) -> Connector_JST:JST_PH_B6B-PH-K_1x06_P2.00mm_Vertical
- J9: footprint (none) -> Connector_PinHeader_1.27mm:PinHeader_2x07_P1.27mm_Vertical_SMD
- L1: footprint (none) -> Capacitor_SMD:C_0402_1005Metric_Pad0.74x0.62mm_HandSolder
- R1, R2, R5, R6, R7, R8, R9: footprint (none) -> Resistor_SMD:R_0402_1005Metric
- SW1: footprint (none) -> Régu:SW_SPST
- SW2: footprint (none) -> Régu:SW_SPDT
Connections:
- net +14.8V: now also R30.1
- net +7.5V: now also C15.2, C18.2, U3.2 (VM), U4.2 (VM)
- net Accel SCL: now also U1.40 (PC8)
- net Accel SDA: now also U1.41 (PC9)
- net GND: now also C34.2, R31.2; no longer U2.12 (SDO/ADDR)
- net INT 1: now also U1.18 (PA4)
- net INT 2: now also U1.19 (PA5)
- net Lidar Output : now also U1.20 (PA6)
- net PWM FWD 1: now also U1.61 (PB8)
- net PWM FWD 2: now also U1.38 (PC6)
- net PWM REV 1: now also U1.60 (PB7)
- net PWM REV 2: now also U1.39 (PC7)
- net PWM_LED1: now also U1.57 (PB4)
- net PWM_LED2: now also U1.58 (PB5)
- net PWM_LED3: now also U1.24 (PB0)
- net PWM_LED4: now also U1.25 (PB1)
- net PWM_LED5: now also U1.59 (PB6)
- net SCL TOF: now also U1.42 (PA8)
- net SDA TOF: now also U1.43 (PA9)
- net SWCLK: now also U1.50 (PA14)
- net SWDIO: now also U1.49 (PA13)
- net UART_Debug_RX: now also U1.17 (PA3)
- net UART_Debug_TX: now also U1.14 (PA2)
- net UART_HC05_RX: now also U1.53 (PC11)
- net UART_HC05_TX: now also U1.52 (PC10)
- net UART_mp3_RX: now also U1.55 (PD2)
- net UART_mp3_TX: now also U1.54 (PC12)
- net USB_DM: now also U1.45 (PA11)
- net USB_DP: now also U1.46 (PA12)
- net XSHUT_1: now also U1.44 (PA10)
- net XSHUT_2: now also U1.51 (PA15)
- net XSHUT_3: now also U1.37 (PB15)
- net XSHUT_4: now also U1.36 (PB14)
- net XSHUT_5: now also U1.34 (PB12)
- net XSHUT_6: now also U1.35 (PB13)
- net XSHUT_7: now also U1.26 (PB2)
- net XSHUT_8: now also U1.62 (PB9)
- net PWM_servo_3: now reaches U1.10 (PC2)
- net PWM_servo_4: now reaches U1.11 (PC3)
- net PWM_servo_5: now reaches U1.12 (PA0)
- net ADC: now reaches U1.13 (PA1)
- net ADC: now also C34.1, R30.2, R31.1
- net STBY_IN: now reaches U1.21 (PA7)
- net PWM_servo_7: now reaches U1.30 (PB10)
- net PWM_servo_8: now reaches U1.33 (PB11)
- net PWM_servo_6: now reaches U1.56 (PB3)
- net PWM_servo_1: now reaches U1.8 (PC0)
- net PWM_servo_2: now reaches U1.9 (PC1)
- no-connect marks 8 -> 16
Other:
- sheet Régulateurs ports: added EN/SYNC_2.8, EN/SYNC_5, EN/SYNC_7.5, PG_2.8, PG_5, PG_7.5, STBY_IN; removed none
- note added: "2.6V"
- note added: "ADC"

Commit message: PCB
Parts:
- removed SW2: SW_SPDT, Régu:SW_SPDT, symbol Switch:SW_SPDT
- added SW2: 472121010111, Régu:SW_Wurth_WS-TOTV_472123020421, symbol New_Library:472121010111
- J7: renamed from J9; MPN (none) -> STLINK-V3MINIE
- L1: footprint Capacitor_SMD:C_0402_1005Metric_Pad0.74x0.62mm_HandSolder -> Inductor_SMD:L_0603_1608Metric
- SW1: MPN (none) -> 430182070816
- U1: renamed from U3; MPN (none) -> ZXBM5210-SP-13
- U2: renamed from U4; MPN (none) -> ZXBM5210-SP-13
- U4: renamed from U2; MPN (none) -> ADXL343BCCZ-RL
- renumbered C14 to C1, C3 to C10, C7 to C11, C4 to C12, C5 to C13, C9 to C14, C10 to C15, C8 to C16, C11 to C17, C15 to C2, C34 to C3, C17 to C4, C18 to C5, C1 to C6, C12 to C7, C2 to C8, C6 to C9, D5 to D1, D3 to D2, D4 to D3, D2 to D4, D1 to D5, J5 to J1, J15 to J2, J6 to J3, J16 to J4, J13 to J5, J12 to J6, R30 to R1, R31 to R2, R5 to R3, R6 to R4, R7 to R5, R1 to R6, R8 to R7, R2 to R8, U1 to U3
Connections:
- net +14.8V: now also SW2.1
- net +3.3V: no longer C15.1
- net GND: now also SW2.G1, SW2.G2; no longer C15.2
- net at J5.2 (Pin_2): now also SW2.2
Other:
- note removed: "USB C pour rasbpi 5V/3A (voir même 4A en pointe)"
- moved on the sheet: C15

Commit message: maj scgematic
Parts:
- SW2: MPN (none) -> 472123020421
Other:
- note added: "Connecteurs"
- note added: "Driver Moteurs"
- note added: "LED de tension"
- note added: "STlink"
- note removed: "Conn"
- note removed: "Moteurs"
- note removed: "Régulateurs"
- moved on the sheet: C1, C2, C3, C4, C5, C7, D1, D2, D3, D4, D5, J2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
