File: hardware/KiCAD/PCB projet ESE/ServoFS90.kicad_sch (KiCad schematic)
At the start: 8 parts, among them J21 Conn_01x03, J22 Conn_01x03, J23 Conn_01x03, J24 Conn_01x03, J25 Conn_01x03, J26 Conn_01x03, J27 Conn_01x03, J28 Conn_01x03

Commit message: maj schematic & pinout CubeIDE
Parts:
- renumbered J21 to J18, J22 to J19, J23 to J20, J24 to J21, J25 to J22, J26 to J23, J27 to J24, J28 to J25
Changed lines of the file:
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@@
 		(dnp no)
 		(fields_autoplaced yes)
-		(property "Reference" "#PWR0114"
+		(property "Reference" "#PWR099"
 			(at 170.18 90.17 0)
 			(effects
@@
 			(project "PCB projet ESE"
 				(path "/61bc2d2d-cd10-4636-b1b1-3d875f78e40b/0d0f6199-fa17-417f-9bc5-2f2c16fc5820"
-					(reference "#PWR0114")
+					(reference "#PWR099")
 					(unit 1)
 				)
@@
 		(dnp no)
 		(fields_autoplaced yes)
-		(property "Reference" "#PWR0118"
+		(property "Reference" "#PWR0103"
 			(at 195.58 90.17 0)
 			(effects
@@
 			(project "PCB projet ESE"
 				(path "/61bc2d2d-cd10-4636-b1b1-3d875f78e40b/0d0f6199-fa17-417f-9bc5-2f2c16fc5820"
-					(reference "#PWR0118")
+					(reference "#PWR0103")
 					(unit 1)
 				)
@@
 		(dnp no)
 		(fields_autoplaced yes)
-		(property "Reference" "#PWR0106"
+		(property "Reference" "#PWR091"
 			(at 119.38 90.17 0)
 			(effects
@@
 			(project "PCB projet ESE"
 				(path "/61bc2d2d-cd10-4636-b1b1-3d875f78e40b/0d0f6199-fa17-417f-9bc5-2f2c16fc5820"
-					(reference "#PWR0106")
+					(reference "#PWR091")
 					(unit 1)
 				)
@@
 		(dnp no)
 		(fields_autoplaced yes)
-		(property "Reference" "#PWR0112"
+		(property "Reference" "#PWR097"
 			(at 167.64 77.47 0)
 			(effects
@@
 			(project "PCB projet ESE"
 				(path "/61bc2d2d-cd10-4636-b1b1-3d875f78e40b/0d0f6199-fa17-417f-9bc5-2f2c16fc5820"
-					(reference "#PWR0112")
+					(reference "#PWR097")
 					(unit 1)
 				)
@@
 		(dnp no)
 		(fields_autoplaced yes)
-		(property "Reference" "#PWR0108"
+		(property "Reference" "#PWR093"
 			(at 142.24 77.47 0)
 			(effects
@@
 			(project "PCB projet ESE"
 				(path "/61bc2d2d-cd10-4636-b1b1-3d875f78e40b/0d0f6199-fa17-417f-9bc5-2f2c16fc5820"
-					(reference "#PWR0108")
+					(reference "#PWR093")
 					(unit 1)
 				)
@@
 		(dnp no)
 		(fields_autoplaced yes)
-		(property "Reference" "#PWR0117"
+		(property "Reference" "#PWR0102"
 			(at 193.04 93.98 0)
 			(effects
@@
 			(project "PCB projet ESE"
 				(path "/61bc2d2d-cd10-4636-b1b1-3d875f78e40b/0d0f6199-fa17-417f-9bc5-2f2c16fc5820"
-					(reference "#PWR0117")
+					(reference "#PWR0102")
 					(unit 1)
 				)
@@
 		(dnp no)
 		(fields_autoplaced yes)
-		(property "Reference" "#PWR0110"
+		(property "Reference" "#PWR095"
 			(at 144.78 90.17 0)
 			(effects
@@
 			(project "PCB projet ESE"
 				(path "/61bc2d2d-cd10-4636-b1b1-3d875f78e40b/0d0f6199-fa17-417f-9bc5-2f2c16fc5820"
-					(reference "#PWR0110")
+					(reference "#PWR095")
 					(unit 1)
 				)
@@
 		(dnp no)
 		(fields_autoplaced yes)
-		(property "Reference" "J21"
+		(property "Reference" "J18"
 			(at 104.14 77.47 0)
 			(effects
@@
 			(project "PCB projet ESE"
 				(path "/61bc2d2d-cd10-4636-b1b1-3d875f78e40b/0d0f6199-fa17-417f-9bc5-2f2c16fc5820"
-					(reference "J21")
+					(reference "J18")
 					(unit 1)
 				)
@@
 		(dnp no)
 		(fields_autoplaced yes)
-		(property "Reference" "#PWR0107"
+		(property "Reference" "#PWR092"
 			(at 119.38 106.68 0)
 			(effects
@@
 			(project "PCB projet ESE"
 				(path "/61bc2d2d-cd10-4636-b1b1-3d875f78e40b/0d0f6199-fa17-417f-9bc5-2f2c16fc5820"
-					(reference "#PWR0107")
+					(reference "#PWR092")
 					(unit 1)
 				)
@@
 		(dnp no)
 		(fields_autoplaced yes)
-		(property "Reference" "J23"
+		(property "Reference" "J20"
 			(at 129.54 77.47 0)
 			(effects
@@
 			(project "PCB projet ESE"
 				(path "/61bc2d2d-cd10-4636-b1b1-3d875f78e40b/0d0f6199-fa17-417f-9bc5-2f2c16fc5820"
-					(reference "J23")
+					(reference "J20")
 					(unit 1)
 				)
@@
 		(dnp no)
 		(fields_autoplaced yes)
-		(property "Reference" "#PWR0111"
+		(property "Reference" "#PWR096"
 			(at 144.78 106.68 0)
 			(effects
@@
 			(project "PCB projet ESE"
 				(path "/61bc2d2d-cd10-4636-b1b1-3d875f78e40b/0d0f6199-fa17-417f-9bc5-2f2c16fc5820"
-					(reference "#PWR0111")
+					(reference "#PWR096")
 					(unit 1)
 				)
@@
 		(dnp no)
 		(fields_autoplaced yes)
-		(property "Reference" "#PWR0119"
+		(property "Reference" "#PWR0104"
 			(at 195.58 106.68 0)
 			(effects
@@
 			(project "PCB projet ESE"
 				(path "/61bc2d2d-cd10-4636-b1b1-3d875f78e40b/0d0f6199-fa17-417f-9bc5-2f2c16fc5820"
-					(reference "#PWR0119")
+					(reference "#PWR0104")
 					(unit 1)
 				)
@@
 		(dnp no)
 		(fields_autoplaced yes)
-		(property "Reference" "J22"
+		(property "Reference" "J19"
 			(at 104.14 93.98 0)
 			(effects
@@
 			(project "PCB projet ESE"
 				(path "/61bc2d2d-cd10-4636-b1b1-3d875f78e40b/0d0f6199-fa17-417f-9bc5-2f2c16fc5820"
-					(reference "J22")
+					(reference "J19")
 					(unit 1)
 				)
@@
 		(dnp no)
 		(fields_autoplaced yes)
-		(property "Reference" "J26"
+		(property "Reference" "J23"
 			(at 154.94 93.98 0)
 			(effects
@@
 			(project "PCB projet ESE"
 				(path "/61bc2d2d-cd10-4636-b1b1-3d875f78e40b/0d0f6199-fa17-417f-9bc5-2f2c16fc5820"
-					(reference "J26")
+					(reference "J23")
 					(unit 1)
 				)
@@
 		(dnp no)
 		(fields_autoplaced yes)
-		(property "Reference" "#PWR0115"
+		(property "Reference" "#PWR0100"
 			(at 170.18 106.68 0)
 			(effects
@@
 			(project "PCB projet ESE"
 				(path "/61bc2d2d-cd10-4636-b1b1-3d875f78e40b/0d0f6199-fa17-417f-9bc5-2f2c16fc5820"
-					(reference "#PWR0115")
+					(reference "#PWR0100")
 					(unit 1)
 				)
@@
 		(dnp no)
 		(fields_autoplaced yes)
-		(property "Reference" "J28"
+		(property "Reference" "J25"
 			(at 180.34 93.98 0)
 			(effects
@@
 			(project "PCB projet ESE"
 				(path "/61bc2d2d-cd10-4636-b1b1-3d875f78e40b/0d0f6199-fa17-417f-9bc5-2f2c16fc5820"
-					(reference "J28")
+					(reference "J25")
 					(unit 1)
 				)
@@
 		(dnp no)
 		(fields_autoplaced yes)
-		(property "Reference" "J25"
+		(property "Reference" "J22"
 			(at 154.94 77.47 0)
 			(effects
@@
 			(project "PCB projet ESE"
 				(path "/61bc2d2d-cd10-4636-b1b1-3d875f78e40b/0d0f6199-fa17-417f-9bc5-2f2c16fc5820"
-					(reference "J25")
+					(reference "J22")
 					(unit 1)
 				)
@@
 		(dnp no)
 		(fields_autoplaced yes)
-		(property "Reference" "#PWR0105"
+		(property "Reference" "#PWR090"
 			(at 116.84 93.98 0)
 			(effects
@@
 			(project "PCB projet ESE"
 				(path "/61bc2d2d-cd10-4636-b1b1-3d875f78e40b/0d0f6199-fa17-417f-9bc5-2f2c16fc5820"
-					(reference "#PWR0105")
+					(reference "#PWR090")
 					(unit 1)
 				)
@@
 		(dnp no)
 		(fields_autoplaced yes)
-		(property "Reference" "#PWR0109"
+		(property "Reference" "#PWR094"
 			(at 142.24 93.98 0)
 			(effects
@@
 			(project "PCB projet ESE"
 				(path "/61bc2d2d-cd10-4636-b1b1-3d875f78e40b/0d0f6199-fa17-417f-9bc5-2f2c16fc5820"
-					(reference "#PWR0109")
+					(reference "#PWR094")
 					(unit 1)
 				)
@@
 		(dnp no)
 		(fields_autoplaced yes)
-		(property "Reference" "#PWR0113"
+		(property "Reference" "#PWR098"
 			(at 167.64 93.98 0)
 			(effects
@@
 			(project "PCB projet ESE"
 				(path "/61bc2d2d-cd10-4636-b1b1-3d875f78e40b/0d0f6199-fa17-417f-9bc5-2f2c16fc5820"
-					(reference "#PWR0113")
+					(reference "#PWR098")
 					(unit 1)
 				)
@@
 		(dnp no)
 		(fields_autoplaced yes)
-		(property "Reference" "J24"
+		(property "Reference" "J21"
 			(at 129.54 93.98 0)
 			(effects
@@
 			(project "PCB projet ESE"
 				(path "/61bc2d2d-cd10-4636-b1b1-3d875f78e40b/0d0f6199-fa17-417f-9bc5-2f2c16fc5820"
-					(reference "J24")
+					(reference "J21")
 					(unit 1)
 				)
@@
 		(dnp no)
 		(fields_autoplaced yes)
-		(property "Reference" "#PWR0104"
+		(property "Reference" "#PWR089"
 			(at 116.84 77.47 0)
 			(effects
@@
 			(project "PCB projet ESE"
 				(path "/61bc2d2d-cd10-4636-b1b1-3d875f78e40b/0d0f6199-fa17-417f-9bc5-2f2c16fc5820"
-					(reference "#PWR0104")
+					(reference "#PWR089")
 					(unit 1)
 				)
@@
 		(dnp no)
 		(fields_autoplaced yes)
-		(property "Reference" "#PWR0116"
+		(property "Reference" "#PWR0101"
 			(at 193.04 77.47 0)
 			(effects
@@
 			(project "PCB projet ESE"
 				(path "/61bc2d2d-cd10-4636-b1b1-3d875f78e40b/0d0f6199-fa17-417f-9bc5-2f2c16fc5820"
-					(reference "#PWR0116")
+					(reference "#PWR0101")
 					(unit 1)
 				)
@@
 		(dnp no)
 		(fields_autoplaced yes)
-		(property "Reference" "J27"
+		(property "Reference" "J24"
 			(at 180.34 77.47 0)
 			(effects
@@
 			(project "PCB projet ESE"
 				(path "/61bc2d2d-cd10-4636-b1b1-3d875f78e40b/0d0f6199-fa17-417f-9bc5-2f2c16fc5820"
-					(reference "J27")
-					(unit 1)
-				)
+					(reference "J24")
+					(unit 1)
+				)
