File: hardware/KiCAD/PCB projet ESE/neopixel.kicad_sch (KiCad schematic)
At the start: 5 parts, among them J16 Conn_01x03, J17 Conn_01x03, J18 Conn_01x03, J19 Conn_01x03, J20 Conn_01x03

Commit message: maj schematic & pinout CubeIDE
Parts:
- removed J17, J19, J20: Conn_01x03, Connector_JST:JST_PH_B3B-PH-K_1x03_P2.00mm_Vertical, symbol Connector_Generic:Conn_01x03
- renumbered J18 to J17
