File: hardware/KiCAD/PCB projet ESE/TOF.kicad_sch (KiCad schematic)
At the start: 10 parts, among them J10 Conn_01x06, J11 Conn_01x06, J12 Conn_01x06, J13 Conn_01x06, J14 Conn_01x06, J15 Conn_01x06, J8 Conn_01x06, J9 Conn_01x06

Commit message: maj schematic & pinout CubeIDE
Parts:
- renumbered R10 to R8, R11 to R9
Connections:
- net +2.8V is gone; now on net +3.3V: J10.5 (Pin_5), J11.5 (Pin_5), J12.5 (Pin_5), J13.5 (Pin_5), J14.5 (Pin_5), J15.5 (Pin_5), J8.5 (Pin_5), J9.5 (Pin_5)
Changed lines of the file:
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@@
 		(dnp no)
 		(fields_autoplaced yes)
-		(property "Reference" "#PWR067"
+		(property "Reference" "#PWR065"
 			(at 140.97 107.95 0)
 			(effects
@@
 			(project "PCB projet ESE"
 				(path "/61bc2d2d-cd10-4636-b1b1-3d875f78e40b/261d7bb0-1163-45ca-901d-11d0cf203b6b"
-					(reference "#PWR067")
+					(reference "#PWR065")
 					(unit 1)
 				)
@@
 		(dnp no)
 		(fields_autoplaced yes)
-		(property "Reference" "#PWR058"
+		(property "Reference" "#PWR056"
 			(at 123.19 106.68 0)
 			(effects
@@
 			(project "PCB projet ESE"
 				(path "/61bc2d2d-cd10-4636-b1b1-3d875f78e40b/261d7bb0-1163-45ca-901d-11d0cf203b6b"
-					(reference "#PWR058")
+					(reference "#PWR056")
 					(unit 1)
 				)
@@
 		(dnp no)
 		(fields_autoplaced yes)
-		(property "Reference" "#PWR059"
+		(property "Reference" "#PWR057"
 			(at 120.65 66.04 0)
 			(effects
@@
 			)
 		)
-		(property "Value" "+2.8V"
+		(property "Value" "+3.3V"
 			(at 120.65 57.15 0)
 			(effects
@@
 			(project "PCB projet ESE"
 				(path "/61bc2d2d-cd10-4636-b1b1-3d875f78e40b/261d7bb0-1163-45ca-901d-11d0cf203b6b"
-					(reference "#PWR059")
+					(reference "#PWR057")
 					(unit 1)
 				)
@@
 		(dnp no)
 		(fields_autoplaced yes)
-		(property "Reference" "#PWR066"
+		(property "Reference" "#PWR064"
 			(at 139.7 88.9 0)
 			(effects
@@
 			)
 		)
-		(property "Value" "+2.8V"
+		(property "Value" "+3.3V"
 			(at 139.7 80.01 0)
 			(effects
@@
 			(project "PCB projet ESE"
 				(path "/61bc2d2d-cd10-4636-b1b1-3d875f78e40b/261d7bb0-1163-45ca-901d-11d0cf203b6b"
-					(reference "#PWR066")
+					(reference "#PWR064")
 					(unit 1)
 				)
@@
 		(dnp no)
 		(fields_autoplaced yes)
-		(property "Reference" "#PWR050"
+		(property "Reference" "#PWR048"
 			(at 104.14 59.69 0)
 			(effects
@@
 			(project "PCB projet ESE"
 				(path "/61bc2d2d-cd10-4636-b1b1-3d875f78e40b/261d7bb0-1163-45ca-901d-11d0cf203b6b"
-					(reference "#PWR050")
+					(reference "#PWR048")
 					(unit 1)
 				)
@@
 		(dnp no)
 		(fields_autoplaced yes)
-		(property "Reference" "R11"
+		(property "Reference" "R9"
 			(at 143.51 110.4899 0)
 			(effects
@@
 			(project "PCB projet ESE"
 				(path "/61bc2d2d-cd10-4636-b1b1-3d875f78e40b/261d7bb0-1163-45ca-901d-11d0cf203b6b"
-					(reference "R11")
+					(reference "R9")
 					(unit 1)
 				)
@@
 		(dnp no)
 		(fields_autoplaced yes)
-		(property "Reference" "#PWR053"
+		(property "Reference" "#PWR051"
 			(at 101.6 66.04 0)
 			(effects
@@
 			)
 		)
-		(property "Value" "+2.8V"
+		(property "Value" "+3.3V"
 			(at 101.6 57.15 0)
 			(effects
@@
 			(project "PCB projet ESE"
 				(path "/61bc2d2d-cd10-4636-b1b1-3d875f78e40b/261d7bb0-1163-45ca-901d-11d0cf203b6b"
-					(reference "#PWR053")
+					(reference "#PWR051")
 					(unit 1)
 				)
@@
 		(dnp no)
 		(fields_autoplaced yes)
-		(property "Reference" "#PWR060"
+		(property "Reference" "#PWR058"
 			(at 120.65 88.9 0)
 			(effects
@@
 			)
 		)
-		(property "Value" "+2.8V"
+		(property "Value" "+3.3V"
 			(at 120.65 80.01 0)
 			(effects
@@
 			(project "PCB projet ESE"
 				(path "/61bc2d2d-cd10-4636-b1b1-3d875f78e40b/261d7bb0-1163-45ca-901d-11d0cf203b6b"
-					(reference "#PWR060")
+					(reference "#PWR058")
 					(unit 1)
 				)
@@
 		(dnp no)
 		(fields_autoplaced yes)
-		(property "Reference" "#PWR052"
+		(property "Reference" "#PWR050"
 			(at 104.14 106.68 0)
 			(effects
@@
 			(project "PCB projet ESE"
 				(path "/61bc2d2d-cd10-4636-b1b1-3d875f78e40b/261d7bb0-1163-45ca-901d-11d0cf203b6b"
-					(reference "#PWR052")
+					(reference "#PWR050")
 					(unit 1)
 				)
@@
 		(dnp no)
 		(fields_autoplaced yes)
-		(property "Reference" "#PWR065"
+		(property "Reference" "#PWR063"
 			(at 139.7 66.04 0)
 			(effects
@@
 			)
 		)
-		(property "Value" "+2.8V"
+		(property "Value" "+3.3V"
 			(at 139.7 57.15 0)
 			(effects
@@
 			(project "PCB projet ESE"
 				(path "/61bc2d2d-cd10-4636-b1b1-3d875f78e40b/261d7bb0-1163-45ca-901d-11d0cf203b6b"
-					(reference "#PWR065")
+					(reference "#PWR063")
 					(unit 1)
 				)
@@
 		(dnp no)
 		(fields_autoplaced yes)
-		(property "Reference" "#PWR062"
+		(property "Reference" "#PWR060"
 			(at 134.62 107.95 0)
 			(effects
@@
 			(project "PCB projet ESE"
 				(path "/61bc2d2d-cd10-4636-b1b1-3d875f78e40b/261d7bb0-1163-45ca-901d-11d0cf203b6b"
-					(reference "#PWR062")
+					(reference "#PWR060")
 					(unit 1)
 				)
@@
 		(dnp no)
 		(fields_autoplaced yes)
-		(property "Reference" "#PWR056"
+		(property "Reference" "#PWR054"
 			(at 123.19 59.69 0)
 			(effects
@@
 			(project "PCB projet ESE"
 				(path "/61bc2d2d-cd10-4636-b1b1-3d875f78e40b/261d7bb0-1163-45ca-901d-11d0cf203b6b"
-					(reference "#PWR056")
+					(reference "#PWR054")
 					(unit 1)
 				)
@@
 		(dnp no)
 		(fields_autoplaced yes)
-		(property "Reference" "#PWR055"
+		(property "Reference" "#PWR053"
 			(at 101.6 113.03 0)
 			(effects
@@
 			)
 		)
-		(property "Value" "+2.8V"
+		(property "Value" "+3.3V"
 			(at 101.6 104.14 0)
 			(effects
@@
 			(project "PCB projet ESE"
 				(path "/61bc2d2d-cd10-4636-b1b1-3d875f78e40b/261d7bb0-1163-45ca-901d-11d0cf203b6b"
-					(reference "#PWR055")
+					(reference "#PWR053")
 					(unit 1)
 				)
@@
 		(dnp no)
 		(fields_autoplaced yes)
-		(property "Reference" "#PWR051"
+		(property "Reference" "#PWR049"
 			(at 104.14 82.55 0)
 			(effects
@@
 			(project "PCB projet ESE"
 				(path "/61bc2d2d-cd10-4636-b1b1-3d875f78e40b/261d7bb0-1163-45ca-901d-11d0cf203b6b"
-					(reference "#PWR051")
+					(reference "#PWR049")
 					(unit 1)
 				)
@@
 		(dnp no)
 		(fields_autoplaced yes)
-		(property "Reference" "#PWR057"
+		(property "Reference" "#PWR055"
 			(at 123.19 82.55 0)
 			(effects
@@
 			(project "PCB projet ESE"
 				(path "/61bc2d2d-cd10-4636-b1b1-3d875f78e40b/261d7bb0-1163-45ca-901d-11d0cf203b6b"
-					(reference "#PWR057")
+					(reference "#PWR055")
 					(unit 1)
 				)
@@
 		(dnp no)
 		(fields_autoplaced yes)
-		(property "Reference" "#PWR061"
+		(property "Reference" "#PWR059"
 			(at 120.65 113.03 0)
 			(effects
@@
 			)
 		)
-		(property "Value" "+2.8V"
+		(property "Value" "+3.3V"
 			(at 120.65 104.14 0)
 			(effects
@@
 			(project "PCB projet ESE"
 				(path "/61bc2d2d-cd10-4636-b1b1-3d875f78e40b/261d7bb0-1163-45ca-901d-11d0cf203b6b"
-					(reference "#PWR061")
+					(reference "#PWR059")
 					(unit 1)
 				)
@@
 		(dnp no)
 		(fields_autoplaced yes)
-		(property "Reference" "R10"
+		(property "Reference" "R8"
 			(at 137.16 110.4899 0)
 			(effects
@@
 			(project "PCB projet ESE"
 				(path "/61bc2d2d-cd10-4636-b1b1-3d875f78e40b/261d7bb0-1163-45ca-901d-11d0cf203b6b"
-					(reference "R10")
+					(reference "R8")
 					(unit 1)
 				)
@@
 		(dnp no)
 		(fields_autoplaced yes)
-		(property "Reference" "#PWR064"
+		(property "Reference" "#PWR062"
 			(at 142.24 82.55 0)
 			(effects
@@
 			(project "PCB projet ESE"
 				(path "/61bc2d2d-cd10-4636-b1b1-3d875f78e40b/261d7bb0-1163-45ca-901d-11d0cf203b6b"
-					(reference "#PWR064")
+					(reference "#PWR062")
 					(unit 1)
 				)
@@
 		(dnp no)
 		(fields_autoplaced yes)
-		(property "Reference" "#PWR063"
+		(property "Reference" "#PWR061"
 			(at 142.24 59.69 0)
 			(effects
@@
 			(project "PCB projet ESE"
 				(path "/61bc2d2d-cd10-4636-b1b1-3d875f78e40b/261d7bb0-1163-45ca-901d-11d0cf203b6b"
-					(reference "#PWR063")
+					(reference "#PWR061")
 					(unit 1)
 				)
@@
 		(dnp no)
 		(fields_autoplaced yes)
-		(property "Reference" "#PWR054"
+		(property "Reference" "#PWR052"
 			(at 101.6 88.9 0)
 			(effects
@@
 			)
 		)
-		(property "Value" "+2.8V"
+		(property "Value" "+3.3V"
 			(at 101.6 80.01 0)
 			(effects
@@
 			(project "PCB projet ESE"
 				(path "/61bc2d2d-cd10-4636-b1b1-3d875f78e40b/261d7bb0-1163-45ca-901d-11d0cf203b6b"
-					(reference "#PWR054")
-					(unit 1)
-				)
+					(reference "#PWR052")
+					(unit 1)
+				)

Commit message: update pcb
Parts:
- J10, J11, J12, J13, J14, J15, J8, J9: footprint Connector_JST:JST_PH_B6B-PH-K_1x06_P2.00mm_Vertical -> Connector_JST:JST_SH_BM06B-SRSS-TB_1x06-1MP_P1.00mm_Vertical
Connections:
- removed net INT: J10.1 (Pin_1), J11.1 (Pin_1), J12.1 (Pin_1), J13.1 (Pin_1), J14.1 (Pin_1), J15.1 (Pin_1), J8.1 (Pin_1), J9.1 (Pin_1)
- new net INT 1: J8.1 (Pin_1)
- new net INT 2: J11.1 (Pin_1)
- new net INT 3: J14.1 (Pin_1)
- new net INT 4: J9.1 (Pin_1)
- new net INT 5: J12.1 (Pin_1)
- new net INT 6: J15.1 (Pin_1)
- new net INT 7: J10.1 (Pin_1)
- new net INT 8: J13.1 (Pin_1)
Changed lines of the file:
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@@
 		)
 	)
-	(hierarchical_label "INT"
+	(hierarchical_label "INT 2"
 		(shape input)
 		(at 116.84 72.39 0)
@@
 		)
 	)
-	(hierarchical_label "INT"
+	(hierarchical_label "INT 4"
 		(shape input)
 		(at 97.79 95.25 0)
@@
 		)
 	)
-	(hierarchical_label "INT"
+	(hierarchical_label "INT 8"
 		(shape input)
 		(at 116.84 119.38 0)
@@
 		)
 	)
-	(hierarchical_label "INT"
+	(hierarchical_label "INT 3"
 		(shape input)
 		(at 135.89 72.39 0)
@@
 		)
 	)
-	(hierarchical_label "INT"
+	(hierarchical_label "INT 5"
 		(shape input)
 		(at 116.84 95.25 0)
@@
 		)
 	)
-	(hierarchical_label "INT"
+	(hierarchical_label "INT 7"
 		(shape input)
 		(at 97.79 119.38 0)
@@
 		)
 	)
-	(hierarchical_label "INT"
+	(hierarchical_label "INT 1"
 		(shape input)
 		(at 97.79 72.39 0)
@@
 		)
 	)
-	(hierarchical_label "INT"
+	(hierarchical_label "INT 6"
 		(shape input)
 		(at 135.89 95.25 0)
@@
 			)
 		)
-		(property "Footprint" "Connector_JST:JST_PH_B6B-PH-K_1x06_P2.00mm_Vertical"
+		(property "Footprint" "Connector_JST:JST_SH_BM06B-SRSS-TB_1x06-1MP_P1.00mm_Vertical"
 			(at 92.71 90.17 0)
 			(effects
@@
 			)
 		)
-		(property "Footprint" "Connector_JST:JST_PH_B6B-PH-K_1x06_P2.00mm_Vertical"
+		(property "Footprint" "Connector_JST:JST_SH_BM06B-SRSS-TB_1x06-1MP_P1.00mm_Vertical"
 			(at 111.76 114.3 0)
 			(effects
@@
 			)
 		)
-		(property "Footprint" "Connector_JST:JST_PH_B6B-PH-K_1x06_P2.00mm_Vertical"
+		(property "Footprint" "Connector_JST:JST_SH_BM06B-SRSS-TB_1x06-1MP_P1.00mm_Vertical"
 			(at 130.81 90.17 0)
 			(effects
@@
 			)
 		)
-		(property "Footprint" "Connector_JST:JST_PH_B6B-PH-K_1x06_P2.00mm_Vertical"
+		(property "Footprint" "Connector_JST:JST_SH_BM06B-SRSS-TB_1x06-1MP_P1.00mm_Vertical"
 			(at 92.71 67.31 0)
 			(effects
@@
 			)
 		)
-		(property "Footprint" "Connector_JST:JST_PH_B6B-PH-K_1x06_P2.00mm_Vertical"
+		(property "Footprint" "Connector_JST:JST_SH_BM06B-SRSS-TB_1x06-1MP_P1.00mm_Vertical"
 			(at 111.76 67.31 0)
 			(effects
@@
 			)
 		)
-		(property "Footprint" "Connector_JST:JST_PH_B6B-PH-K_1x06_P2.00mm_Vertical"
+		(property "Footprint" "Connector_JST:JST_SH_BM06B-SRSS-TB_1x06-1MP_P1.00mm_Vertical"
 			(at 92.71 114.3 0)
 			(effects
@@
 			)
 		)
-		(property "Footprint" "Connector_JST:JST_PH_B6B-PH-K_1x06_P2.00mm_Vertical"
+		(property "Footprint" "Connector_JST:JST_SH_BM06B-SRSS-TB_1x06-1MP_P1.00mm_Vertical"
 			(at 111.76 90.17 0)
 			(effects
@@
 			)
 		)
-		(property "Footprint" "Connector_JST:JST_PH_B6B-PH-K_1x06_P2.00mm_Vertical"
+		(property "Footprint" "Connector_JST:JST_SH_BM06B-SRSS-TB_1x06-1MP_P1.00mm_Vertical"
 			(at 130.81 67.31 0)
 			(effects

Commit message: v1 PCB
Parts:
- removed J10, J13: Conn_01x06, Connector_JST:JST_SH_BM06B-SRSS-TB_1x06-1MP_P1.00mm_Vertical, symbol Connector_Generic:Conn_01x06
- renumbered J8 to J10, J9 to J11, J11 to J12, J12 to J13
Connections:
- net +3.3V: now also J10.1 (Pin_1), J11.1 (Pin_1), J12.1 (Pin_1), J13.1 (Pin_1), J14.1 (Pin_1), J15.1 (Pin_1); no longer J10.5 (Pin_5), J11.5 (Pin_5), J12.5 (Pin_5), J13.5 (Pin_5), J14.5 (Pin_5), J15.5 (Pin_5)
- net GND: now also J10.2 (Pin_2), J11.2 (Pin_2), J12.2 (Pin_2), J13.2 (Pin_2), J14.2 (Pin_2), J15.2 (Pin_2); no longer J10.6 (Pin_6), J11.6 (Pin_6), J12.6 (Pin_6), J13.6 (Pin_6), J14.6 (Pin_6), J15.6 (Pin_6)
- net INT 1: now also J10.5 (Pin_5); no longer J10.1 (Pin_1)
- net INT 2: now also J12.5 (Pin_5); no longer J12.1 (Pin_1)
- net INT 3: now also J14.5 (Pin_5); no longer J14.1 (Pin_1)
- net INT 4: now also J11.5 (Pin_5); no longer J11.1 (Pin_1)
- net INT 5: now also J13.5 (Pin_5); no longer J13.1 (Pin_1)
- net INT 6: now also J15.5 (Pin_5); no longer J15.1 (Pin_1)
- net SCL TOF: now also J10.3 (Pin_3), J11.3 (Pin_3), J12.3 (Pin_3), J13.3 (Pin_3), J14.3 (Pin_3), J15.3 (Pin_3); no longer J10.2 (Pin_2), J11.2 (Pin_2), J12.2 (Pin_2), J13.2 (Pin_2), J14.2 (Pin_2), J15.2 (Pin_2)
- net XSHUT_1: now also J10.6 (Pin_6); no longer J10.3 (Pin_3)
- net XSHUT_2: now also J12.6 (Pin_6); no longer J12.3 (Pin_3)
- net XSHUT_3: now also J14.6 (Pin_6); no longer J14.3 (Pin_3)
- net XSHUT_4: now also J11.6 (Pin_6); no longer J11.3 (Pin_3)
- net XSHUT_5: now also J13.6 (Pin_6); no longer J13.3 (Pin_3)
- net XSHUT_6: now also J15.6 (Pin_6); no longer J15.3 (Pin_3)
Other:
- note added: "1 3.3V 2 GND 3 SCL 4 SDA 5 INT 6 Xhut"
- note added: "18mm x 12 mm"
