File: hardware/KiCAD/PCB projet ESE/Régulateurs.kicad_sch (KiCad schematic)
At the start: 33 parts

Commit message: v1 PCB
Parts:
- removed C19, C29, C31: 22u, Capacitor_SMD:C_Elec_5x5.4, symbol Device:C_Small
- removed C21, C23, C25: 0.1u, Capacitor_SMD:C_0402_1005Metric, symbol Device:C_Small
- removed C27: 15p, Capacitor_SMD:C_0402_1005Metric, symbol Device:C_Small
- removed L3: 4.7u, Inductor_SMD:L_0603_1608Metric, symbol Device:L_Small
- removed MP2: ~, Régu:TSOT23-8, symbol Regulateur:MP1475
- removed R11, R13: 100k, Resistor_SMD:R_0402_1005Metric, symbol Device:R_Small
- removed R15: 20, Resistor_SMD:R_0402_1005Metric, symbol Device:R_Small
- removed R17: 16k, Resistor_SMD:R_0402_1005Metric, symbol Device:R_Small
- removed R19: 7.68k, Resistor_SMD:R_0402_1005Metric, symbol Device:R_Small
- removed R21: 40.2k, Resistor_SMD:R_0402_1005Metric, symbol Device:R_Small
- C20: renamed from C18; footprint Capacitor_SMD:C_Elec_5x5.4 -> Capacitor_SMD:C_1206_3216Metric
- C25: renamed from C28; footprint Capacitor_SMD:C_Elec_5x5.4 -> Capacitor_SMD:C_0603_1608Metric
- C26: renamed from C30; footprint Capacitor_SMD:C_Elec_5x5.4 -> Capacitor_SMD:C_0603_1608Metric
- renumbered C20 to C21, C24 to C23, C26 to C24, C32 to C27, C33 to C28, R12 to R11, R14 to R12, R16 to R13, R18 to R14, R20 to R15
Other:
- note removed: "Les LABELS (IN, VCC...) ne sont pas forcément exact, il faut les vérifier"

Commit message: BOM
Parts:
- C21, C22, C23: value 0.1u -> 100n
- L2: value 4.7u -> 4u7
- R14: value 7.68k -> 7k68
- R15: value 40.2k -> 40k2
Changed lines of the file:
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@@
 			)
 		)
-		(property "Value" "0.1u"
+		(property "Value" "100n"
 			(at 88.9 35.5662 0)
 			(effects
@@
 			)
 		)
-		(property "Value" "7.68k"
+		(property "Value" "7k68"
 			(at 101.6 54.61 0)
 			(effects
@@
 			)
 		)
-		(property "Value" "0.1u"
+		(property "Value" "100n"
 			(at 50.8 40.6462 0)
 			(effects
@@
 			)
 		)
-		(property "Value" "0.1u"
+		(property "Value" "100n"
 			(at 52.07 33.0262 0)
 			(effects
@@
 			)
 		)
-		(property "Value" "4.7u"
+		(property "Value" "4u7"
 			(at 109.22 31.242 90)
 			(effects
@@
 			)
 		)
-		(property "Value" "40.2k"
+		(property "Value" "40k2"
 			(at 113.538 52.324 90)
 			(effects

Commit message: maj inductance 4.7uH
Parts:
- L2: footprint Inductor_SMD:L_0603_1608Metric -> Régu:74404054068
Changed lines of the file:
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@@
 			)
 		)
-		(property "Footprint" "Inductor_SMD:L_0603_1608Metric"
+		(property "Footprint" "Régu:74404054068"
 			(at 109.22 33.02 0)
 			(effects

Commit message: maj C25 & C26
Parts:
- C25, C26: footprint Capacitor_SMD:C_0603_1608Metric -> Capacitor_SMD:C_0805_2012Metric
Changed lines of the file:
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@@
 			)
 		)
-		(property "Footprint" "Capacitor_SMD:C_0603_1608Metric"
+		(property "Footprint" "Capacitor_SMD:C_0805_2012Metric"
 			(at 127 30.48 0)
 			(effects
@@
 			)
 		)
-		(property "Footprint" "Capacitor_SMD:C_0603_1608Metric"
+		(property "Footprint" "Capacitor_SMD:C_0805_2012Metric"
 			(at 118.11 30.48 0)
 			(effects
