File: hardware/KiCAD/PCB_Projet_ESE/PCB projet ESE.kicad_sch (KiCad schematic)
At the start: 56 parts, among them J1 Conn_01x06, J16 Conn_01x04, J2 Conn_01x04, J3 Conn_01x06, J4 Conn_01x03, J7 Conn_01x04, J8 Conn_01x02, J9 Conn_ST_STDC14, SW1 SW_SPST, SW2 472121010111, U1 ZXBM5210-SP, U2 ZXBM5210-SP, U3 STM32G474RETx, U4 ADXL343

Commit message: review pcb
Connections:
- net 5V_Rpi: now reaches C29.1, C30.1, D5.2 (A2), F2.1, J16.2 (Pin_2)
Changed lines of the file:
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@@
+		)
+	)
+	(label "5V_Rpi"
+		(at 77.47 186.69 0)
+		(effects
+			(font
+				(size 1.27 1.27)
+			)
+			(justify left bottom)
 		)
 	)
