File: hardware/KiCAD/PCB_Projet_ESE/PCB projet ESE.kicad_pcb (KiCad board)
At the start: 4 copper layers, 53 x 46 mm, 82 parts, among them J1 Conn_01x06, J10 Conn_01x06, J11 Conn_01x06, J12 Conn_01x06, J13 Conn_01x06, J14 Conn_01x06, J15 Conn_01x06, J16 Conn_01x04, J2 Conn_01x04, J3 Conn_01x06, J4 Conn_01x03, J7 Conn_01x04, J8 Conn_01x02, J9 Conn_ST_STDC14, SW1 SW_SPST, SW2 472121010111, U1 ZXBM5210-SP, U2 ZXBM5210-SP, U3 STM32G474RETx, U4 ADXL343

Commit message: review pcb
Parts:
- F2: value 3.3A -> 1A
- TP1: renamed from PWM REV 2
- TP2: renamed from PWM FWD 2
- TP3: renamed from PWM REV 1
- TP4: renamed from ACCEL SCL
- TP5: renamed from ACCEL SDA
- TP6: renamed from PWM FWD 1
- moved TP4 2.15 mm to (101.1, 80.4)
- moved TP5 0.41 mm to (103.0, 79.7)
Connections:
- net Net-(D5-A2) renamed /5V_Rpi
- J10 pad MP: GND -> (no net)
- J11 pad MP: GND -> (no net)
- J12 pad MP: GND -> (no net)
- J13 pad MP: GND -> (no net)
- J14 pad MP: GND -> (no net)
- J15 pad MP: GND -> (no net)
- J2 pad MP: GND -> (no net)
Routing:
- net UART_mp3_RX: track 24.6 -> 28.3 mm
- net Net-(MP1-SW): track 12.3 -> 14.8 mm, vias 6 -> 5
- net NRST: track 33.9 -> 36.4 mm, vias 4 -> 3
- net UART_Pi_Zero_RX: track 30.2 -> 31.9 mm
- net PWM FWD 2: track 19.9 -> 21.2 mm
- net GND: track 87.6 -> 86.4 mm, vias 120 -> 132
- net SWCLK: track 15.0 -> 15.6 mm
- net +5V: vias 10 -> 14
- added copper zone on B.Cu, net +5V

Commit message: gerbers
Parts:
- Accel SCL: renamed from TP4
- Accel SDA: renamed from TP5
- PWM FWD 1: renamed from TP6
- PWM FWD 2: renamed from TP2
- PWM REV 1: renamed from TP3
- PWM REV 2: renamed from TP1
Connections:
- J10 pad MP: (no net) -> GND
- J11 pad MP: (no net) -> GND
- J12 pad MP: (no net) -> GND
- J13 pad MP: (no net) -> GND
- J14 pad MP: (no net) -> GND
- J15 pad MP: (no net) -> GND
- J2 pad MP: (no net) -> GND
Routing:
- net GND: track 86.4 -> 88.4 mm, vias 132 -> 133
