File: hardware/KiCAD/PCB_AMPLI/PCB_AMPLI.kicad_pcb (KiCad board)
At the start: 2 copper layers, 22 parts, among them J1 Conn_01x02, J2 Conn_01x02, J3 Conn_01x02, J4 Conn_01x02, J5 Conn_01x02, J6 Conn_01x02, J7 Conn_01x02, J8 Conn_01x02, SW1 SW_SPDT, SW2 SW_SPDT

Commit message: sch v2 ampli
Parts:
- added C6: 10u, Capacitor_SMD:C_0603_1608Metric, F.Cu at (141.2, 93.0)
- added D1: GREEN_LED, LED_SMD:LED_0603_1608Metric, F.Cu at (141.3, 80.2)
- added D2: RED_LED, LED_SMD:LED_0603_1608Metric, F.Cu at (141.3, 82.8)
- added D3: BLUE_LED, LED_SMD:LED_0603_1608Metric, F.Cu at (141.3, 85.4)
- added J9: Conn_01x02, Connector_PinHeader_2.54mm:PinHeader_1x02_P2.54mm_Vertical, F.Cu at (157.6, 67.5)
- added R4: 5k, Resistor_SMD:R_0402_1005Metric, F.Cu at (129.9, 95.2)
- added R5: 5k, Resistor_SMD:R_0402_1005Metric, F.Cu at (129.9, 97.2)
- added R6: 1k5, Resistor_SMD:R_0402_1005Metric, F.Cu at (129.9, 99.2)
- added SW3: SW_SPDT, Personal:450406020024, F.Cu at (123.2, 99.6)
- C1: value 1u -> 100n; footprint Capacitor_SMD:C_0603_1608Metric -> Capacitor_SMD:C_0402_1005Metric
- C4: value 100n -> 1u; footprint Capacitor_SMD:C_0402_1005Metric -> Capacitor_SMD:C_0603_1608Metric
- R1: value 1k5 -> 1k8
- R2: value 5k -> 1k
- R3: value 5k -> 510
- moved J1 70.6 mm to (120.4, 67.5), turned to 0 degrees
- moved SW1 70.5 mm to (123.2, 80.0)
- moved J2 67.0 mm to (125.1, 67.5), turned to 0 degrees
- moved J3 63.9 mm to (129.7, 67.5), turned to 0 degrees
- moved J4 61.3 mm to (134.4, 67.5), turned to 0 degrees
- moved H2 51.4 mm to (132.4, 84.3)
- moved SW2 50.7 mm to (123.2, 89.8)
- moved H1 47.9 mm to (132.4, 76.4)
- moved U1 42.3 mm to (140.8, 75.7)
- moved J5 35.9 mm to (139.0, 67.5), turned to 0 degrees
- moved J6 33.5 mm to (143.7, 67.5), turned to 0 degrees
- moved J8 32.4 mm to (153.0, 67.5), turned to 0 degrees
- moved J7 32.3 mm to (148.3, 67.5), turned to 0 degrees
- moved C1 13.1 mm to (137.8, 79.9)
- moved R1 12.0 mm to (129.9, 89.3)
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Connections:
- C1 pad 1: PVDD -> GND
- C1 pad 2: GND -> I2C_VDD_SW
- C2 pad 1: VDD -> Net-(U1-IN2)
- C2 pad 2: GND -> IN2
- C4 pad 1: Net-(U1-IN2) -> PVDD_SW
- C4 pad 2: IN2 -> GND
- C7 pad 1: GND -> VDD
- C7 pad 2: I2C_VDD -> GND
- J1 pad 1: IN2 -> IN1
- J2 pad 1: IN1 -> OUTA
- J3 pad 1: I2C_VDD -> PVDD
- J4 pad 1: VDD -> IN2
- J6 pad 1: OUTA -> VDD
- J8 pad 1: PVDD -> I2C_VDD
- R1 pad 1: VDD -> PVDD
- R1 pad 2: FAULT -> Net-(D1-A)
- R2 pad 2: SDA -> Net-(D2-A)
- R3 pad 1: SCL -> VDD
- R3 pad 2: I2C_VDD -> Net-(D3-A)
- SW2 pad 2: I2C_VDD -> I2C_VDD_SW
- U1 pad 10: PVDD -> PVDD_SW
- U1 pad 4: I2C_VDD -> I2C_VDD_SW

Commit message: pcb ampli final 1.0
Parts:
- removed J1, J5, J6, J7, J8, J9: Conn_01x02, Connector_PinHeader_2.54mm:PinHeader_1x02_P2.54mm_Vertical
- added J10: Conn_01x04, Connector_PinHeader_2.54mm:PinHeader_1x04_P2.54mm_Vertical, F.Cu at (163.0, 121.0)
- J3, J4: value Conn_01x02 -> Conn_01x04; footprint Connector_PinHeader_2.54mm:PinHeader_1x02_P2.54mm_Vertical -> Connector_PinHeader_2.54mm:PinHeader_1x04_P2.54mm_Vertical
- moved J3 65.2 mm to (167.0, 121.0), turned to 90 degrees
- moved SW1 58.8 mm to (168.8, 117.2)
- moved J2 58.5 mm to (170.0, 105.0)
- moved H1 57.8 mm to (177.5, 112.5), turned to 90 degrees
- moved J4 54.3 mm to (143.8, 121.0), turned to 90 degrees
- moved SW2 45.2 mm to (159.3, 117.2)
- moved C2 36.5 mm to (164.1, 107.2)
- moved U1 36.2 mm to (159.1, 107.0)
- moved C3 34.4 mm to (164.1, 106.2)
- moved SW3 31.8 mm to (149.8, 117.2)
- moved C1 31.6 mm to (154.1, 107.0)
- moved C4 31.1 mm to (163.9, 109.3), turned to -90 degrees
- moved C7 30.1 mm to (162.1, 103.7)
- moved H2 29.5 mm to (141.0, 112.5), turned to 90 degrees
- moved C6 29.2 mm to (165.5, 109.3), turned to -90 degrees
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Connections:
- J2 pad 2: GND -> OUTB
- J3 pad 1: PVDD -> IN1
- J4 pad 1: IN2 -> SCL
- J4 pad 2: GND -> SDA
- SW1 pad 1: I2C_VDD -> I2C_VDD_SW
Routing:
- net SCL: track 0.00 -> 24.3 mm, vias 0 -> 1
- net IN1: track 0.00 -> 23.0 mm, vias 0 -> 2
- net ADR: track 0.00 -> 22.4 mm
- net PVDD: track 0.00 -> 21.5 mm
- net FAULT: track 0.00 -> 21.4 mm, vias 0 -> 1
- net SDA: track 0.00 -> 20.2 mm, vias 0 -> 1
- net IN2: track 0.00 -> 19.3 mm
- net I2C_VDD: track 0.00 -> 18.6 mm, vias 0 -> 1
- net GND: track 0.00 -> 17.5 mm, vias 0 -> 54
- net OUTA: track 0.00 -> 17.0 mm, vias 0 -> 1
- net I2C_VDD_SW: track 0.00 -> 16.9 mm, vias 0 -> 5
- net VDD: track 0.00 -> 10.9 mm, vias 0 -> 7
- net OUTB: track 0.00 -> 9.59 mm, vias 0 -> 1
- net PVDD_SW: track 0.00 -> 6.83 mm, vias 0 -> 4
- net Net-(U1-BIAS): track 0.00 -> 2.27 mm
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- added copper zone on B.Cu, net GND
- added copper zone on F.Cu, net GND
- added copper zone on In1.Cu, net GND
- added copper zone on In2.Cu, net I2C_VDD_SW
- added copper zone on In2.Cu, net PVDD_SW
- added copper zone on In2.Cu, net VDD
Other:
- board outline added: 46.5 x 20.8 mm
- copper layers 2 -> 4
- board text added: "+"
- board text added: "-"
- board text added: "3.0V ≤ VDD/PVDD ≤ 5.5V 1.8V ≤ I2C_VDD ≤ 5.5V"
- board text added: "FAULT"
- board text added: "GND"
- board text added: "I2C"
- board text added: "I2C VDD"
- board text added: "I2C_VDD"
- board text added: "INT1"
- board text added: "INT2"
- board text added: "OUT"
- board text added: "PROJET ESE V. FERNANDES"
- board text added: "PVDD"
- board text added: "SCL"
- board text added: "SDA"
- board text added: "SW1 : ADR = I2C_VDD | GND SW2 : I2C_VDD = I2C_VDD | VDD SW3 : PVDD = PVDD | VDD"
- board text added: "VDD"
