File: hardware/KiCAD/PCB_Projet_ESE_v2/Régulateurs.kicad_sch (KiCad schematic)
At the start: 18 parts

Commit message: Schematic done for PCB v2
Parts:
- renumbered C20 to C34, C21 to C35, C22 to C36, C23 to C37, C24 to C38, C25 to C39, C26 to C40, C27 to C41, C28 to C42, R10 to R15, R11 to R16, R12 to R17, R13 to R18, R14 to R19, R15 to R20
Connections:
- net PG_51 renamed PG
Changed lines of the file:
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@@
 		)
 	)
-	(hierarchical_label "PG_51"
+	(hierarchical_label "PG"
 		(shape input)
 		(at 41.91 82.55 180)
@@
 		(dnp no)
 		(fields_autoplaced yes)
-		(property "Reference" "R10"
+		(property "Reference" "R15"
 			(at 50.8 86.3599 0)
 			(effects
@@
 			(project "PCB_Projet_ESE_v2"
 				(path "/e93b439b-eb98-463a-8161-b748b1434139/1255fbdd-dd20-42db-b7f6-2aa7912bc741"
-					(reference "R10")
+					(reference "R15")
 					(unit 1)
 				)
@@
 		(dnp no)
 		(fields_autoplaced yes)
-		(property "Reference" "C27"
+		(property "Reference" "C41"
 			(at 180.34 69.8562 0)
 			(effects
@@
 			(project "PCB_Projet_ESE_v2"
 				(path "/e93b439b-eb98-463a-8161-b748b1434139/1255fbdd-dd20-42db-b7f6-2aa7912bc741"
-					(reference "C27")
+					(reference "C41")
 					(unit 1)
 				)
@@
 		(dnp no)
 		(fields_autoplaced yes)
-		(property "Reference" "#FLG03"
+		(property "Reference" "#FLG05"
 			(at 151.13 74.295 0)
 			(effects
@@
 			(project "PCB_Projet_ESE_v2"
 				(path "/e93b439b-eb98-463a-8161-b748b1434139/1255fbdd-dd20-42db-b7f6-2aa7912bc741"
-					(reference "#FLG03")
+					(reference "#FLG05")
 					(unit 1)
 				)
@@
 		(on_board yes)
 		(dnp no)
-		(property "Reference" "C23"
+		(property "Reference" "C37"
 			(at 101.6 73.152 0)
 			(effects
@@
 			(project "PCB_Projet_ESE_v2"
 				(path "/e93b439b-eb98-463a-8161-b748b1434139/1255fbdd-dd20-42db-b7f6-2aa7912bc741"
-					(reference "C23")
+					(reference "C37")
 					(unit 1)
 				)
@@
 		(on_board yes)
 		(dnp no)
-		(property "Reference" "R14"
+		(property "Reference" "R19"
 			(at 114.3 91.44 0)
 			(effects
@@
 			(project "PCB_Projet_ESE_v2"
 				(path "/e93b439b-eb98-463a-8161-b748b1434139/1255fbdd-dd20-42db-b7f6-2aa7912bc741"
-					(reference "R14")
+					(reference "R19")
 					(unit 1)
 				)
@@
 		(on_board yes)
 		(dnp no)
-		(property "Reference" "C21"
+		(property "Reference" "C35"
 			(at 63.5 77.4762 0)
 			(effects
@@
 			(project "PCB_Projet_ESE_v2"
 				(path "/e93b439b-eb98-463a-8161-b748b1434139/1255fbdd-dd20-42db-b7f6-2aa7912bc741"
-					(reference "C21")
+					(reference "C35")
 					(unit 1)
 				)
@@
 		(dnp no)
 		(fields_autoplaced yes)
-		(property "Reference" "C22"
+		(property "Reference" "C36"
 			(at 64.77 69.8562 0)
 			(effects
@@
 			(project "PCB_Projet_ESE_v2"
 				(path "/e93b439b-eb98-463a-8161-b748b1434139/1255fbdd-dd20-42db-b7f6-2aa7912bc741"
-					(reference "C22")
+					(reference "C36")
 					(unit 1)
 				)
@@
 		(on_board yes)
 		(dnp no)
-		(property "Reference" "#PWR069"
+		(property "Reference" "#PWR075"
 			(at 113.03 102.87 0)
 			(effects
@@
 			(project "PCB_Projet_ESE_v2"
 				(path "/e93b439b-eb98-463a-8161-b748b1434139/1255fbdd-dd20-42db-b7f6-2aa7912bc741"
-					(reference "#PWR069")
+					(reference "#PWR075")
 					(unit 1)
 				)
@@
 		(on_board yes)
 		(dnp no)
-		(property "Reference" "C26"
+		(property "Reference" "C40"
 			(at 141.732 68.834 0)
 			(effects
@@
 			(project "PCB_Projet_ESE_v2"
 				(path "/e93b439b-eb98-463a-8161-b748b1434139/1255fbdd-dd20-42db-b7f6-2aa7912bc741"
-					(reference "C26")
+					(reference "C40")
 					(unit 1)
 				)
@@
 		(on_board yes)
 		(dnp no)
-		(property "Reference" "#PWR066"
+		(property "Reference" "#PWR072"
 			(at 57.15 59.69 0)
 			(effects
@@
 			(project "PCB_Projet_ESE_v2"
 				(path "/e93b439b-eb98-463a-8161-b748b1434139/1255fbdd-dd20-42db-b7f6-2aa7912bc741"
-					(reference "#PWR066")
+					(reference "#PWR072")
 					(unit 1)
 				)
@@
 		(dnp no)
 		(fields_autoplaced yes)
-		(property "Reference" "C28"
+		(property "Reference" "C42"
 			(at 212.09 69.8562 0)
 			(effects
@@
 			(project "PCB_Projet_ESE_v2"
 				(path "/e93b439b-eb98-463a-8161-b748b1434139/1255fbdd-dd20-42db-b7f6-2aa7912bc741"
-					(reference "C28")
+					(reference "C42")
 					(unit 1)
 				)
@@
 		(on_board yes)
 		(dnp no)
-		(property "Reference" "R13"
+		(property "Reference" "R18"
 			(at 100.076 84.328 90)
 			(effects
@@
 			(project "PCB_Projet_ESE_v2"
 				(path "/e93b439b-eb98-463a-8161-b748b1434139/1255fbdd-dd20-42db-b7f6-2aa7912bc741"
-					(reference "R13")
+					(reference "R18")
 					(unit 1)
 				)
@@
 		(on_board yes)
 		(dnp no)
-		(property "Reference" "#PWR068"
+		(property "Reference" "#PWR074"
 			(at 85.09 96.52 0)
 			(effects
@@
 			(project "PCB_Projet_ESE_v2"
 				(path "/e93b439b-eb98-463a-8161-b748b1434139/1255fbdd-dd20-42db-b7f6-2aa7912bc741"
-					(reference "#PWR068")
+					(reference "#PWR074")
 					(unit 1)
 				)
@@
 		(dnp no)
 		(fields_autoplaced yes)
-		(property "Reference" "#PWR074"
+		(property "Reference" "#PWR080"
 			(at 196.85 86.36 0)
 			(effects
@@
 			(project "PCB_Projet_ESE_v2"
 				(path "/e93b439b-eb98-463a-8161-b748b1434139/1255fbdd-dd20-42db-b7f6-2aa7912bc741"
-					(reference "#PWR074")
+					(reference "#PWR080")
 					(unit 1)
 				)
@@
 		(dnp no)
 		(fields_autoplaced yes)
-		(property "Reference" "#PWR071"
+		(property "Reference" "#PWR077"
 			(at 151.13 74.93 0)
 			(effects
@@
 			(project "PCB_Projet_ESE_v2"
 				(path "/e93b439b-eb98-463a-8161-b748b1434139/1255fbdd-dd20-42db-b7f6-2aa7912bc741"
-					(reference "#PWR071")
+					(reference "#PWR077")
 					(unit 1)
 				)
@@
 		(dnp no)
 		(fields_autoplaced yes)
-		(property "Reference" "#PWR076"
+		(property "Reference" "#PWR082"
 			(at 223.52 72.39 0)
 			(effects
@@
 			(project "PCB_Projet_ESE_v2"
 				(path "/e93b439b-eb98-463a-8161-b748b1434139/1255fbdd-dd20-42db-b7f6-2aa7912bc741"
-					(reference "#PWR076")
+					(reference "#PWR082")
 					(unit 1)
 				)
@@
 		(dnp no)
 		(fields_autoplaced yes)
-		(property "Reference" "#PWR075"
+		(property "Reference" "#PWR081"
 			(at 209.55 83.82 0)
 			(effects
@@
 			(project "PCB_Projet_ESE_v2"
 				(path "/e93b439b-eb98-463a-8161-b748b1434139/1255fbdd-dd20-42db-b7f6-2aa7912bc741"
-					(reference "#PWR075")
+					(reference "#PWR081")
 					(unit 1)
 				)
@@
 		(dnp no)
 		(fields_autoplaced yes)
-		(property "Reference" "C20"
+		(property "Reference" "C34"
 			(at 54.61 69.8562 0)
 			(effects
@@
 			(project "PCB_Projet_ESE_v2"
 				(path "/e93b439b-eb98-463a-8161-b748b1434139/1255fbdd-dd20-42db-b7f6-2aa7912bc741"
-					(reference "C20")
+					(reference "C34")
 					(unit 1)
 				)
@@
 		(on_board yes)
 		(dnp no)
-		(property "Reference" "R12"
+		(property "Reference" "R17"
 			(at 95.25 64.516 90)
 			(effects
@@
 			(project "PCB_Projet_ESE_v2"
 				(path "/e93b439b-eb98-463a-8161-b748b1434139/1255fbdd-dd20-42db-b7f6-2aa7912bc741"
-					(reference "R12")
+					(reference "R17")
 					(unit 1)
 				)
@@
 		(on_board yes)
 		(dnp no)
-		(property "Reference" "R15"
+		(property "Reference" "R20"
 			(at 125.73 89.916 90)
 			(effects
@@
 			(project "PCB_Projet_ESE_v2"
 				(path "/e93b439b-eb98-463a-8161-b748b1434139/1255fbdd-dd20-42db-b7f6-2aa7912bc741"
-					(reference "R15")
+					(reference "R20")
 					(unit 1)
 				)
@@
 		(on_board yes)
 		(dnp no)
-		(property "Reference" "C25"
+		(property "Reference" "C39"
 			(at 132.588 69.088 0)
 			(effects
@@
 			(project "PCB_Projet_ESE_v2"
 				(path "/e93b439b-eb98-463a-8161-b748b1434139/1255fbdd-dd20-42db-b7f6-2aa7912bc741"
-					(reference "C25")
+					(reference "C39")
 					(unit 1)
 				)
@@
 		(on_board yes)
 		(dnp no)
-		(property "Reference" "C24"
+		(property "Reference" "C38"
 			(at 125.73 77.47 90)
 			(effects
@@
 			(project "PCB_Projet_ESE_v2"
 				(path "/e93b439b-eb98-463a-8161-b748b1434139/1255fbdd-dd20-42db-b7f6-2aa7912bc741"
-					(reference "C24")
+					(reference "C38")
 					(unit 1)
 				)
@@
 		(on_board yes)
 		(dnp no)
-		(property "Reference" "#PWR067"
+		(property "Reference" "#PWR073"
 			(at 60.96 91.44 0)
 			(effects
@@
 			(project "PCB_Projet_ESE_v2"
 				(path "/e93b439b-eb98-463a-8161-b748b1434139/1255fbdd-dd20-42db-b7f6-2aa7912bc741"
-					(reference "#PWR067")
+					(reference "#PWR073")
 					(unit 1)
 				)
@@
 		(dnp no)
 		(fields_autoplaced yes)
-		(property "Reference" "#PWR065"
+		(property "Reference" "#PWR071"
 			(at 40.64 77.47 0)
 			(effects
@@
 			(project "PCB_Projet_ESE_v2"
 				(path "/e93b439b-eb98-463a-8161-b748b1434139/1255fbdd-dd20-42db-b7f6-2aa7912bc741"
-					(reference "#PWR065")
+					(reference "#PWR071")
 					(unit 1)
 				)
@@
 		(on_board yes)
 		(dnp no)
-		(property "Reference" "#PWR070"
+		(property "Reference" "#PWR076"
 			(at 130.81 55.88 0)
 			(effects
@@
 			(project "PCB_Projet_ESE_v2"
 				(path "/e93b439b-eb98-463a-8161-b748b1434139/1255fbdd-dd20-42db-b7f6-2aa7912bc741"
-					(reference "#PWR070")
+					(reference "#PWR076")
 					(unit 1)
 				)
@@
 		(on_board yes)
 		(dnp no)
-		(property "Reference" "#PWR073"
+		(property "Reference" "#PWR079"
 			(at 177.8 80.01 0)
 			(effects
@@
 			(project "PCB_Projet_ESE_v2"
 				(path "/e93b439b-eb98-463a-8161-b748b1434139/1255fbdd-dd20-42db-b7f6-2aa7912bc741"
-					(reference "#PWR073")
+					(reference "#PWR079")
 					(unit 1)
 				)
@@
 		(on_board yes)
 		(dnp no)
-		(property "Reference" "R11"
+		(property "Reference" "R16"
 			(at 52.07 77.47 0)
 			(effects
@@
 			(project "PCB_Projet_ESE_v2"
 				(path "/e93b439b-eb98-463a-8161-b748b1434139/1255fbdd-dd20-42db-b7f6-2aa7912bc741"
-					(reference "R11")
+					(reference "R16")
 					(unit 1)
 				)
@@
 		(dnp no)
 		(fields_autoplaced yes)
-		(property "Reference" "#PWR072"
+		(property "Reference" "#PWR078"
 			(at 171.45 72.39 0)
 			(effects
@@
 			(project "PCB_Projet_ESE_v2"
 				(path "/e93b439b-eb98-463a-8161-b748b1434139/1255fbdd-dd20-42db-b7f6-2aa7912bc741"
-					(reference "#PWR072")
-					(unit 1)
-				)
+					(reference "#PWR078")
+					(unit 1)
+				)

Commit message: routage en cours
Parts:
- C41, C42: footprint Capacitor_SMD:C_0603_1608Metric -> Capacitor_SMD:C_0402_1005Metric
Changed lines of the file:
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@@
 			)
 		)
-		(property "Footprint" "Capacitor_SMD:C_0603_1608Metric"
+		(property "Footprint" "Capacitor_SMD:C_0402_1005Metric"
 			(at 177.8 71.12 0)
 			(effects
@@
 			)
 		)
-		(property "Footprint" "Capacitor_SMD:C_0603_1608Metric"
+		(property "Footprint" "Capacitor_SMD:C_0402_1005Metric"
 			(at 209.55 71.12 0)
 			(effects
