File: hardware/KiCAD/PCB_Projet_ESE_v2/PCB_Projet_ESE_v2.kicad_pcb (KiCad board)
At the start: 6 copper layers, 45 x 45 mm, 203 parts, among them J1 Conn_01x06, J10 Conn_ST_STDC14, J2 Conn_01x06, J4 Conn_01x03, J5 Conn_01x04, J6 Conn_01x04, J9 Conn_01x02, SW1 SW_SPST, SW3 SW_SPST, SW4 SW_SPDT, SW5 SW_SPDT, U1 ZXBM5210-SP, U16 MCP1802x-xx02xOT, U2 ZXBM5210-SP, U3 NCS210, U4 NCS210, U5 STM32G474RETx, U6 ADXL343, Y1 Crystal_GND24_Small

Commit message: TOF polling
Parts:
- moved TP9 0.34 mm to (77.4, 85.3)
Routing:
- net GND: track 147.2 -> 162.6 mm, vias 104 -> 118
- net +3.3V: track 76.3 -> 84.0 mm, vias 26 -> 29
- net +5V: track 50.5 -> 53.9 mm, vias 21 -> 23
- net VREF_+3.3V: track 35.2 -> 37.3 mm, vias 7 -> 8
- net +7.4V: track 30.0 -> 31.9 mm, vias 10 -> 11
- net /5V_Rpi: track 6.04 -> 7.74 mm, vias 7 -> 6
- net ADC_Moteur_2: track 23.1 -> 24.7 mm
- net TOF_1_XSHUT: track 47.3 -> 48.5 mm
- net UART_Pi_Zero_TX: track 7.81 -> 8.85 mm, vias 0 -> 1
- net TOF_2_XSHUT: track 43.2 -> 44.2 mm
- net 30%: track 8.37 -> 9.05 mm, vias 1 -> 2
- net TOF_5_XSHUT: track 37.2 -> 36.6 mm
- net SWCLK: track 16.6 -> 16.1 mm

Commit message: PCB V2 routage v2 finished
Parts:
- removed SW3: SW_SPST, mylib:SW_SPST
- added D1: BLUE_LED_0402, LED_SMD:LED_0402_1005Metric, F.Cu at (83.9, 58.5)
- added D21: BLUE_LED_0402, LED_SMD:LED_0402_1005Metric, F.Cu at (83.9, 59.5)
- added D22: BLUE_LED_0402, LED_SMD:LED_0402_1005Metric, F.Cu at (83.9, 60.5)
- added D23: BLUE_LED_0402, LED_SMD:LED_0402_1005Metric, F.Cu at (83.9, 63.5)
- added D24: BLUE_LED_0402, LED_SMD:LED_0402_1005Metric, F.Cu at (83.9, 62.5)
- added D25: BLUE_LED_0402, LED_SMD:LED_0402_1005Metric, F.Cu at (83.9, 61.5)
- added H2: MountingHole_Pad, mylib:Pad_traversant_M1, F.Cu at (69.2, 97.8)
- added H3: MountingHole_Pad, mylib:Pad_traversant_M1, F.Cu at (85.8, 97.8)
- added H4: MountingHole_Pad, mylib:Pad_traversant_M1, F.Cu at (69.2, 57.2)
- added R25: 200, Resistor_SMD:R_0201_0603Metric, F.Cu at (85.8, 58.9)
- added R26: 200, Resistor_SMD:R_0201_0603Metric, F.Cu at (85.8, 59.8)
- added R27: 200, Resistor_SMD:R_0201_0603Metric, F.Cu at (85.8, 60.7)
- added R28: 200, Resistor_SMD:R_0201_0603Metric, F.Cu at (85.8, 63.4)
- added R39: 200, Resistor_SMD:R_0201_0603Metric, F.Cu at (85.8, 62.5)
- added R40: 200, Resistor_SMD:R_0201_0603Metric, F.Cu at (85.8, 61.6)
- added SW2: ~, mylib:WS-TASV SMT Tact Switch 3.0 x 2.6 mm, F.Cu at (62.7, 68.0)
- C51, J5, R51, R52, R53, R55, R57, R58, R61, R62, R65, R66, R68: moved to F.Cu
- C9: moved to B.Cu
- H1: footprint MountingHole:MountingHole_2.2mm_M2_Pad_Via -> mylib:Pad_traversant_M1
- R23, R24: value 300 -> 1k
- R54: value 98k8 -> 100k; footprint Resistor_SMD:R_0402_1005Metric -> Resistor_SMD:R_0201_0603Metric; moved to F.Cu
- R56, R67: value 79k6 -> 78k7; footprint Resistor_SMD:R_0402_1005Metric -> Resistor_SMD:R_0201_0603Metric; moved to F.Cu
- R69: value 98k8 -> 100k; footprint Resistor_SMD:R_0402_1005Metric -> Resistor_SMD:R_0201_0603Metric
- R72: footprint Resistor_SMD:R_0201_0603Metric -> Resistor_SMD:R_0402_1005Metric
- SW1: value SW_SPST -> ~; footprint mylib:SW_SPST -> mylib:WS-TASV SMT Tact Switch 3.0 x 2.6 mm; moved to F.Cu
- TP1, TP10, TP11, TP2: footprint TestPoint:TestPoint_Pad_D2.0mm -> TestPoint:TestPoint_Pad_D1.0mm; moved to B.Cu
- TP3, TP4, TP5, TP6, TP7, TP8, TP9: footprint TestPoint:TestPoint_Pad_D2.0mm -> TestPoint:TestPoint_Pad_D1.0mm
- U10, U11, U12, U13, U14, U15: footprint mylib:JST_SH_6_Vertical -> mylib:Wurth_Vertical_6_pos_0.8mm
- U7, U9: footprint mylib:JST_SH_4_Vertical -> mylib:Wurth_Vertical_4_pos_0.8mm
- U8: footprint mylib:JST_SH_4_Vertical -> mylib:Wurth_Vertical_4_pos_0.8mm; moved to F.Cu
- moved U9 32.8 mm to (58.0, 71.6), turned to 180 degrees
- moved C7 32.2 mm to (57.8, 72.8), turned to 90 degrees
- moved H1 21.9 mm to (85.8, 57.2)
- moved R63 19.3 mm to (78.0, 66.2), turned to -90 degrees
- moved R65 18.6 mm to (76.8, 66.5), turned to 0 degrees
- moved R64 17.8 mm to (78.8, 65.8), turned to 90 degrees
- moved R66 17.6 mm to (77.0, 67.3), turned to 180 degrees
- moved C65 17.3 mm to (76.8, 68.2), turned to 180 degrees
- moved R62 16.4 mm to (82.0, 66.2), turned to 90 degrees
- moved C66 16.1 mm to (79.7, 66.0), turned to 90 degrees
- moved C67 15.6 mm to (81.1, 66.0), turned to 90 degrees
- moved TP2 15.1 mm to (79.4, 76.9), turned to 180 degrees
- moved U7 15.1 mm to (67.0, 60.5), turned to 135 degrees
- moved R58 14.2 mm to (66.8, 71.2), turned to -135 degrees
- moved R61 14.2 mm to (82.8, 66.2), turned to -90 degrees
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Connections:
- SW1 pad 2: GND -> NRST
Routing:
- net GND: track 162.6 -> 215.9 mm, vias 118 -> 181
- net IN+: track 26.0 -> 62.9 mm, vias 5 -> 11
- net VREF_+3.3V: track 37.3 -> 57.6 mm, vias 8 -> 9
- net TOF_6_GPIO: track 33.6 -> 52.7 mm, vias 2 -> 3
- net TOF_SCL: track 59.8 -> 41.0 mm, vias 11 -> 7
- net PG: track 0.00 -> 17.6 mm, vias 0 -> 4
- net +7.4V: track 31.9 -> 49.2 mm, vias 11 -> 12
- net TOF_SDA: track 57.7 -> 40.6 mm, vias 9 -> 8
- net Net-(C38-Pad1): track 2.23 -> 14.3 mm, vias 0 -> 3
- net UART_mp3_RX: track 27.8 -> 39.8 mm, vias 2 -> 5
- net AMPLI_SDA: track 44.5 -> 32.7 mm
- net TOF_1_XSHUT: track 48.5 -> 38.2 mm, vias 5 -> 2
- net TOF_3_GPIO: track 24.0 -> 32.8 mm, vias 2 -> 4
- net TOF_2_GPIO: track 23.2 -> 31.6 mm, vias 2 -> 4
- net ACCEL_INT1: track 11.5 -> 19.4 mm, vias 0 -> 2
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- added copper zone on In6.Cu, net +3.3V
- added copper zone on In5.Cu, net GND
- added copper zone on B.Cu, net IN+
- added copper zone on F.Cu, net Net-(J9-Pin_2)
- removed copper zone on In3.Cu, net +3.3V
- removed copper zone on B.Cu, net /5V_Rpi
- removed copper zone on In3.Cu, net IN+
- removed copper zone on In3.Cu, net Net-(J9-Pin_2)
Other:
- copper layers 6 -> 8

Commit message: ordered PCB v2
Routing:
- net /5V_Rpi: track 8.93 -> 9.92 mm, vias 0 -> 4
- added copper zone on B.Cu, net /5V_Rpi
Other:
- board text added: "ACCEL INT1"
- board text added: "ACCEL INT2"
- board text added: "ACCEL SCL"
- board text added: "ACCEL SDA"
- board text added: "ADC Bat"
- board text added: "ADC Mot 1"
- board text added: "ADC Mot 2"
- board text added: "ESE V.F"
- board text added: "Mot 1 REV"
- board text added: "Mot 2 FWD"
- board text added: "Mot 2 REV"
