File: hardware/KiCAD/PCB_Projet_ESE_v2/PCB_Projet_ESE_v2.kicad_sch (KiCad schematic)
At the start: 91 parts, among them J1 Conn_01x06, J10 Conn_ST_STDC14, J2 Conn_01x06, J4 Conn_01x03, J5 Conn_01x04, J6 Conn_01x04, J9 Conn_01x02, SW1 SW_SPST, SW3 SW_SPST, SW4 SW_SPDT, SW5 SW_SPDT, U1 ZXBM5210-SP, U2 ZXBM5210-SP, U3 NCS210, U4 NCS210, U5 STM32G474RETx, U6 ADXL343, Y1 Crystal_GND24_Small

Commit message: routage en cours
Parts:
- removed D1: D_TVS_Small, Diode_SMD:D_SOD-523, symbol Device:D_TVS_Small
- added C69, C70, C71, C72: 100n, Capacitor_SMD:C_0402_1005Metric, symbol Device:C_Small
- added D20: ~, Diode_SMD:D_SOD-523, symbol my_lib:VESD05A1-02V-G3-08
- added D7, D8: YELLOW_LED, mylib:wurth_155060YS75300, symbol Device:LED
- added R23, R24: 300, Resistor_SMD:R_0402_1005Metric, symbol Device:R_Small
- added R73, R74: 4k7, Resistor_SMD:R_0402_1005Metric, symbol Device:R_Small
- C22, C30, C31: footprint Capacitor_SMD:C_0603_1608Metric -> Capacitor_SMD:C_0402_1005Metric
- J5, J6: footprint Connector_JST:JST_PH_B4B-PH-K_1x04_P2.00mm_Vertical -> Connector_THT_Wurth:J_Wurth_WR-WTB_62000411722
- R10: value 5k6 -> 16k
- R11: value 240 -> 39
- R12: value 2k9 -> 2k7
- R13: value 1k65 -> 1k6
- R14: value 800 -> 820
- R9: value 20k -> 56k
- SW4, SW5: footprint mylib:472123010111 -> mylib:SW_Wurth_WS-TOTV_472123020421; symbol Switch:SW_SPDT -> New_Library:472121010111; Actuator Length (Value) (mm) (none) -> 10.4; Bushing Length (Value) (mm) (none) -> 9.0; Manufacturer (none) -> Wurth Elektronik; Manufacturer URL (none) -> https://www.we-online.com; Match Code (none) -> WS-TOTV; Mounting Technology (none) -> THT; Part Number (none) -> 472121010111; Published Date (none) -> 20250626; Schematic (none) -> SPDT; Switching Function (none) -> ON-ON
- renumbered Mot_1_REV to TP8, Mot_1_FWD to TP9
Connections:
- net +3.3V: now also R73.1, R74.1
- net 5V_Rpi: now also D20.2 (A2)
- net AMPLI_SCL: now also U5.38 (PC6), R74.2; no longer U5.40 (PC8)
- net AMPLI_SDA: now also U5.39 (PC7), R73.2; no longer U5.41 (PC9)
- net GND: now also U5.61 (PB8), C69.1, C70.2, C71.1, C72.2, D20.1 (A1), D7.1 (K), D8.1 (K)
- net Mode_1: now also R23.1
- net Mode_2: now also R24.1
- net Moteur_1_OUT+: now also C69.2
- net Moteur_1_OUT-: now also C70.1
- net Moteur_2_OUT+: now also C71.2
- net Moteur_2_OUT-: now also C72.1
- net TOF_1_XSHUT: now also U5.44 (PA10); no longer U5.19 (PA5)
- net TOF_2_XSHUT: now also U5.33 (PB11); no longer U5.21 (PA7)
- net TOF_3_GPIO: now also U5.60 (PB7); no longer U5.59 (PB6)
- net TOF_3_XSHUT: now also U5.21 (PA7); no longer U5.44 (PA10)
- net TOF_4_GPIO: now also U5.62 (PB9); no longer U5.60 (PB7)
- net TOF_4_XSHUT: now also U5.19 (PA5); no longer U5.23 (PC5)
- net TOF_5_GPIO: now also U5.59 (PB6); no longer U5.62 (PB9)
- net TOF_5_XSHUT: now also U5.23 (PC5); no longer U5.33 (PB11)
- net TOF_SCL: now also U5.40 (PC8); no longer U5.38 (PC6)
- net TOF_SDA: now also U5.41 (PC9); no longer U5.39 (PC7)
- new net: D8.2 (A), R24.2
- new net: D7.2 (A), R23.2
- no-connect marks 7 -> 10
Other:
- added sheet Battery_Monitoring (Battery_Monitoring.kicad_sch)
- moved on the sheet: C6

Commit message: TOF polling
Parts:
- D7, D8: MPN VLMB1501-GS08 -> 155060YS75300
- R1, R2: MPN (none) -> WSK25123L000DEA
- R23, R24: value 300 -> 1k
Other:
- note removed: "A CHANGER SCHELATIC DIODE TVS ONE SIDED"
Changed lines of the file:
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@@
 		)
 	)
-	(text "A CHANGER SCHELATIC DIODE TVS ONE SIDED"
-		(exclude_from_sim no)
-		(at 95.758 187.706 0)
-		(effects
-			(font
-				(size 1.27 1.27)
-				(thickness 0.254)
-				(bold yes)
-				(italic yes)
-				(color 0 255 0 1)
-			)
-		)
-	)
 	(text "1.65V"
 		(exclude_from_sim no)
@@
 			)
 		)
-		(property "Datasheet" "https://www.vishay.com/docs/82554/vlmo1500.pdf"
+		(property "Datasheet" "https://www.we-online.com/components/products/datasheet/155060YS75300.pdf"
 			(at 156.21 5.08 0)
 			(effects
@@
 			)
 		)
-		(property "MPN" "VLMB1501-GS08 "
+		(property "MPN" "155060YS75300"
 			(at 156.21 5.08 0)
 			(effects
@@
 			)
 		)
-		(property "Datasheet" "~"
+		(property "Datasheet" "https://www.vishay.com/docs/30108/wsk2512.pdf"
 			(at 73.66 78.74 0)
 			(effects
@@
 			)
 		)
+		(property "MPN" "WSK25123L000DEA "
+			(at 73.66 78.74 0)
+			(effects
+				(font
+					(size 1.27 1.27)
+				)
+				(hide yes)
+			)
+		)
 		(pin "2"
 		)
@@
 			)
 		)
-		(property "Value" "300"
+		(property "Value" "1k"
 			(at 147.32 17.78 90)
 			(effects
@@
 			)
 		)
-		(property "Datasheet" "~"
+		(property "Datasheet" "https://www.vishay.com/docs/30108/wsk2512.pdf"
 			(at 78.74 35.56 0)
 			(effects
@@
 			)
 		)
+		(property "MPN" "WSK25123L000DEA "
+			(at 78.74 35.56 0)
+			(effects
+				(font
+					(size 1.27 1.27)
+				)
+				(hide yes)
+			)
+		)
 		(pin "2"
 		)
@@
 			)
 		)
-		(property "Value" "300"
+		(property "Value" "1k"
 			(at 149.86 2.54 90)
 			(effects
@@
 			)
 		)
-		(property "Datasheet" "https://www.vishay.com/docs/82554/vlmo1500.pdf"
+		(property "Datasheet" "http://we-online.com/components/products/datasheet/155060YS75300.pdf"
 			(at 153.67 20.32 0)
 			(effects
@@
 			)
 		)
-		(property "MPN" "VLMB1501-GS08 "
+		(property "MPN" "155060YS75300"
 			(at 153.67 20.32 0)
 			(effects

Commit message: PCB V2 routage v2 finished
Parts:
- removed SW1, SW3: SW_SPST, mylib:SW_SPST, symbol Switch:SW_SPST
- added SW1, SW2: ~, mylib:WS-TASV SMT Tact Switch 3.0 x 2.6 mm, symbol my_lib:WS-TASV_SMT_Tact_Switch_3.0_x_2.6_mm
- H1: footprint MountingHole:MountingHole_2.2mm_M2_Pad_Via -> mylib:Pad_traversant_M1
- H2, H3, H4: footprint MountingHole:MountingHole_3.2mm_M3_Pad_Via -> mylib:Pad_traversant_M1
- TP1, TP10, TP11, TP2, TP3, TP4, TP5, TP6, TP7, TP8, TP9: footprint TestPoint:TestPoint_Pad_D2.0mm -> TestPoint:TestPoint_Pad_D1.0mm
- U7, U8, U9: footprint mylib:JST_SH_4_Vertical -> mylib:Wurth_Vertical_4_pos_0.8mm
Connections:
- net GND: now also SW1.3, SW1.4, SW1.5, SW1.6 (GND), SW2.3, SW2.4, SW2.5, SW2.6 (GND)
- net INT_BTN: now also SW2.1, SW2.2
- net NRST: now also SW1.1, SW1.2

Commit message: ordered PCB v2
Parts:
- R11: value 39 -> 620
Other:
- note added: "///////////////////"
- note added: "150060BS75003"
Changed lines of the file:
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@@
 		)
 	)
+	(text "///////////////////"
+		(exclude_from_sim no)
+		(at 235.204 127.254 0)
+		(effects
+			(font
+				(size 1.27 1.27)
+				(thickness 0.254)
+				(bold yes)
+				(italic yes)
+				(color 255 0 255 1)
+			)
+		)
+	)
 	(text "1.65V"
 		(exclude_from_sim no)
@@
 		)
 	)
+	(text "150060BS75003	"
+		(exclude_from_sim no)
+		(at 235.204 129.794 0)
+		(effects
+			(font
+				(size 1.27 1.27)
+			)
+		)
+	)
 	(junction
 		(at 179.07 25.4)
@@
 			)
 		)
-		(property "Value" "39"
+		(property "Value" "620"
 			(at 234.95 120.65 90)
 			(effects
