File: hardware/KiCAD/PCB_Projet_ESE_v2/Battery_Monitoring.kicad_sch (KiCad schematic)
At the start: 73 parts, among them U16 MCP1802x-xx02xOT

Commit message: PCB V2 routage v2 finished
Parts:
- R54, R69: value 98k8 -> 100k; footprint Resistor_SMD:R_0402_1005Metric -> Resistor_SMD:R_0201_0603Metric
- R56, R67: value 79k6 -> 78k7; footprint Resistor_SMD:R_0402_1005Metric -> Resistor_SMD:R_0201_0603Metric
- R72: footprint Resistor_SMD:R_0201_0603Metric -> Resistor_SMD:R_0402_1005Metric
Other:
- note added: "CRCW02015K23FNED 0201"
- note added: "CRCW020178K7FNED 0201"
- note removed: "0201"
- note removed: "CRCW02015K23FNED"
- note removed: "TNPW040279K6BEED"
- note removed: "TNPW060398K8BEEA"
Changed lines of the file:
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@@
 	(text "CRCW0201100KJNED 0201"
 		(exclude_from_sim no)
-		(at 40.386 71.628 0)
+		(at 36.322 78.994 0)
 		(effects
 			(font
@@
 		)
 	)
-	(text "CRCW020146K4FNED 0201"
+	(text "CRCW0201100KJNED 0201"
 		(exclude_from_sim no)
-		(at 35.56 153.924 0)
+		(at 81.026 171.196 0)
 		(effects
 			(font
@@
 		)
 	)
-	(text "CRCW020120K0JNED 0201"
+	(text "CRCW020146K4FNED 0201"
 		(exclude_from_sim no)
-		(at 34.29 113.284 0)
+		(at 35.56 155.194 0)
 		(effects
 			(font
@@
 		)
 	)
-	(text "TNPW040279K6BEED\n"
+	(text "CRCW020120K0JNED 0201"
 		(exclude_from_sim no)
-		(at 33.274 128.27 0)
+		(at 34.29 113.284 0)
 		(effects
 			(font
@@
 		)
 	)
-	(text "CRCW020120K0JNED 0201"
+	(text "CRCW020178K7FNED 0201"
 		(exclude_from_sim no)
-		(at 78.486 101.346 0)
+		(at 35.306 130.556 0)
 		(effects
 			(font
@@
 		)
 	)
-	(text "0201\n"
+	(text "CRCW020120K0JNED 0201"
 		(exclude_from_sim no)
-		(at 50.546 64.008 0)
+		(at 78.486 101.346 0)
 		(effects
 			(font
 				(size 1.27 1.27)
-				(color 0 255 0 1)
+				(color 255 0 0 1)
 			)
 		)
@@
 		)
 	)
-	(text "CRCW02015K23FNED"
+	(text "CRCW02015K23FNED 0201"
 		(exclude_from_sim no)
-		(at 103.124 72.898 0)
+		(at 102.87 77.978 0)
 		(effects
 			(font
@@
 	(text "CRCW020130K0JNED 0201"
 		(exclude_from_sim no)
-		(at 37.338 179.578 0)
+		(at 33.782 180.848 0)
 		(effects
 			(font
@@
 		)
 	)
-	(text "CRCW020120K0JNED 0201"
+	(text "CRCW0201100KJNED 0201"
 		(exclude_from_sim no)
-		(at 39.116 138.938 0)
+		(at 35.814 102.616 0)
 		(effects
 			(font
@@
 		)
 	)
-	(text "TNPW020111K0BEED 0201"
+	(text "CRCW020120K0JNED 0201"
 		(exclude_from_sim no)
-		(at 34.29 88.138 0)
+		(at 39.116 138.938 0)
 		(effects
 			(font
@@
 		)
 	)
-	(text "TNPW060398K8BEEA"
+	(text "TNPW020111K0BEED 0201"
 		(exclude_from_sim no)
-		(at 33.02 102.87 0)
+		(at 34.29 88.138 0)
 		(effects
 			(font
@@
 		)
 	)
-	(text "CRCW02015K23FNED"
+	(text "CRCW02015K23FNED 0201"
 		(exclude_from_sim no)
-		(at 38.1 64.008 0)
+		(at 37.338 59.944 0)
 		(effects
 			(font
@@
 		)
 	)
-	(text "0201\n"
+	(text "CRCW020120K0JNED 0201"
 		(exclude_from_sim no)
-		(at 115.57 72.898 0)
+		(at 33.528 164.846 0)
 		(effects
 			(font
 				(size 1.27 1.27)
-				(color 0 255 0 1)
+				(color 255 0 0 1)
 			)
 		)
 	)
-	(text "CRCW020120K0JNED 0201"
+	(text "5V"
 		(exclude_from_sim no)
-		(at 40.386 165.1 0)
+		(at 153.67 13.97 0)
 		(effects
 			(font
 				(size 1.27 1.27)
-				(color 255 0 0 1)
 			)
 		)
 	)
-	(text "5V"
+	(text "CRCW020178K7FNED 0201"
 		(exclude_from_sim no)
-		(at 153.67 13.97 0)
+		(at 77.47 144.272 0)
 		(effects
 			(font
 				(size 1.27 1.27)
+				(color 255 0 0 1)
 			)
 		)
@@
 	(text "CRCW020120K0JNED 0201"
 		(exclude_from_sim no)
-		(at 79.502 153.416 0)
+		(at 76.2 156.972 0)
 		(effects
 			(font
@@
 			)
 		)
-		(property "Value" "98k8"
+		(property "Value" "100k"
 			(at 60.96 171.4499 0)
 			(effects
@@
 			)
 		)
-		(property "Footprint" "Resistor_SMD:R_0402_1005Metric"
+		(property "Footprint" "Resistor_SMD:R_0201_0603Metric"
 			(at 58.42 170.18 0)
 			(effects
@@
 			)
 		)
-		(property "Value" "79k6"
+		(property "Value" "78k7"
 			(at 22.86 125.7299 0)
 			(effects
@@
 			)
 		)
-		(property "Footprint" "Resistor_SMD:R_0402_1005Metric"
+		(property "Footprint" "Resistor_SMD:R_0201_0603Metric"
 			(at 20.32 124.46 0)
 			(effects
@@
 			)
 		)
-		(property "Footprint" "Resistor_SMD:R_0201_0603Metric"
+		(property "Footprint" "Resistor_SMD:R_0402_1005Metric"
 			(at 85.09 72.39 0)
 			(effects
@@
 			)
 		)
-		(property "Value" "98k8"
+		(property "Value" "100k"
 			(at 22.86 100.3299 0)
 			(effects
@@
 			)
 		)
-		(property "Footprint" "Resistor_SMD:R_0402_1005Metric"
+		(property "Footprint" "Resistor_SMD:R_0201_0603Metric"
 			(at 20.32 99.06 0)
 			(effects
@@
 			)
 		)
-		(property "Value" "79k6"
+		(property "Value" "78k7"
 			(at 60.96 146.0499 0)
 			(effects
@@
 			)
 		)
-		(property "Footprint" "Resistor_SMD:R_0402_1005Metric"
+		(property "Footprint" "Resistor_SMD:R_0201_0603Metric"
 			(at 58.42 144.78 0)
 			(effects

Commit message: ordered PCB v2
Other:
- note added: "vert jaune orange TLMO1100 ambre rouge super rouge"
- note removed: "vert jaune orange TMO1100 ambre rouge super rouge"
Changed lines of the file:
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@@
 		)
 	)
-	(text "vert\njaune \norange TMO1100\nambre \nrouge\nsuper rouge"
+	(text "vert\njaune \norange TLMO1100\nambre \nrouge\nsuper rouge"
 		(exclude_from_sim no)
 		(at 99.06 27.94 0)

Commit message: Finish README
Other:
- moved on the sheet: C58, C59, C60, C61, C62, C63, C64, C65, C66, C67, C68, R51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
